File: PassiveLiFiTag/LiFi_Receiver_X/LiFi_Receiver.kicad_sch (KiCad schematic)
At the start: 0 parts

Commit message: Added some small peripherals and voltage supplies/decoupling caps
Other:
- removed sheet MSP430FR5994
Changed lines of the file:
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@@
   )
   (text "RH/T Sensors" (at 38.1 102.87 0)
-    (effects (font (face "Ubuntu") (size 3 3)) (justify left bottom))
+    (effects (font (face "Ubuntu") (size 4 4)) (justify left bottom))
   )
   (text "/Peripherals\n" (at 120.65 177.8 0)
-    (effects (font (face "Ubuntu") (size 3 3)) (justify left bottom))
+    (effects (font (face "Ubuntu") (size 4 4)) (justify left bottom))
   )
   (text "LiFi Comm Rx\n" (at 204.47 88.9 0)
-    (effects (font (face "Ubuntu") (size 3 3)) (justify left bottom))
+    (effects (font (face "Ubuntu") (size 4 4)) (justify left bottom))
   )
   (text "MSPFR5994\n" (at 127 107.95 0)
-    (effects (font (face "Ubuntu") (size 5 5)) (justify left bottom))
+    (effects (font (face "Ubuntu") (size 4 4)) (justify left bottom))
   )
   (text "RF Backscatter\n" (at 123.19 35.56 0)
-    (effects (font (face "Ubuntu") (size 3 3)) (justify left bottom))
+    (effects (font (face "Ubuntu") (size 4 4)) (justify left bottom))
   )
   (text "Buttons" (at 120.65 171.45 0)
-    (effects (font (face "Ubuntu") (size 3 3)) (justify left bottom))
+    (effects (font (face "Ubuntu") (size 4 4)) (justify left bottom))
   )
   (text "LiFi Power \n\n" (at 208.28 128.27 0)
-    (effects (font (face "Ubuntu") (size 3 3)) (justify left bottom))
+    (effects (font (face "Ubuntu") (size 4 4)) (justify left bottom))
   )
   (symbol (lib_id "Graphic:SYM_Arrow_XLarge") (at 96.52 93.98 0) (unit 1)
     (in_bom no) (on_board no) (dnp no) (fields_autoplaced)
     (property "Reference" "#SYM1" (at 96.52 91.694 0)
-      (effects (font (size 1 1)) hide)
+      (effects (font (size 1.27 1.27)) hide)
     )
     (property "Value" "SYM_Arrow_XLarge" (at 96.52 96.012 0)
-      (effects (font (size 1 1)) hide)
+      (effects (font (size 1.27 1.27)) hide)
     )
     (property "Footprint" "" (at 96.52 93.98 0)
-      (effects (font (size 1 1)) hide)
+      (effects (font (size 1.27 1.27)) hide)
     )
     (property "Datasheet" "~" (at 96.52 93.98 0)
-      (effects (font (size 1 1)) hide)
+      (effects (font (size 1.27 1.27)) hide)
     )
     (property "Sim.Enable" "0" (at 96.52 93.98 0)
-      (effects (font (size 1 1)) hide)
+      (effects (font (size 1.27 1.27)) hide)
     )
     (instances
@@
     (in_bom no) (on_board no) (dnp no) (fields_autoplaced)
     (property "Reference" "#SYM4" (at 138.684 57.15 0)
-      (effects (font (size 1 1)) hide)
+      (effects (font (size 1.27 1.27)) hide)
     )
     (property "Value" "SYM_Arrow_XLarge" (at 143.002 57.15 0)
-      (effects (font (size 1 1)) hide)
+      (effects (font (size 1.27 1.27)) hide)
     )
     (property "Footprint" "" (at 140.97 57.15 0)
-      (effects (font (size 1 1)) hide)
+      (effects (font (size 1.27 1.27)) hide)
     )
     (property "Datasheet" "~" (at 140.97 57.15 0)
-      (effects (font (size 1 1)) hide)
+      (effects (font (size 1.27 1.27)) hide)
     )
     (property "Sim.Enable" "0" (at 140.97 57.15 0)
-      (effects (font (size 1 1)) hide)
+      (effects (font (size 1.27 1.27)) hide)
     )
     (instances
@@
     (in_bom no) (on_board no) (dnp no)
     (property "Reference" "#SYM2" (at 90.17 104.394 0)
-      (effects (font (size 1 1)) hide)
+      (effects (font (size 1.27 1.27)) hide)
     )
     (property "Value" "SYM_Arrow_XLarge" (at 90.17 108.712 0)
-      (effects (font (size 1 1)) hide)
+      (effects (font (size 1.27 1.27)) hide)
     )
     (property "Footprint" "" (at 90.17 106.68 0)
-      (effects (font (size 1 1)) hide)
+      (effects (font (size 1.27 1.27)) hide)
     )
     (property "Datasheet" "~" (at 90.17 106.68 0)
-      (effects (font (size 1 1)) hide)
+      (effects (font (size 1.27 1.27)) hide)
     )
     (property "Sim.Enable" "0" (at 90.17 106.68 0)
-      (effects (font (size 1 1)) hide)
+      (effects (font (size 1.27 1.27)) hide)
     )
     (instances
@@
     (in_bom no) (on_board no) (dnp no)
     (property "Reference" "#SYM3" (at 182.88 84.074 0)
-      (effects (font (size 1 1)) hide)
+      (effects (font (size 1.27 1.27)) hide)
     )
     (property "Value" "SYM_Arrow_XLarge" (at 182.88 88.392 0)
-      (effects (font (size 1 1)) hide)
+      (effects (font (size 1.27 1.27)) hide)
     )
     (property "Footprint" "" (at 182.88 86.36 0)
-      (effects (font (size 1 1)) hide)
+      (effects (font (size 1.27 1.27)) hide)
     )
     (property "Datasheet" "~" (at 182.88 86.36 0)
-      (effects (font (size 1 1)) hide)
+      (effects (font (size 1.27 1.27)) hide)
     )
     (property "Sim.Enable" "0" (at 182.88 86.36 0)
-      (effects (font (size 1 1)) hide)
+      (effects (font (size 1.27 1.27)) hide)
     )
     (instances
@@
     (in_bom no) (on_board no) (dnp no) (fields_autoplaced)
     (property "Reference" "#SYM6" (at 146.304 146.05 0)
-      (effects (font (size 1 1)) hide)
+      (effects (font (size 1.27 1.27)) hide)
     )
     (property "Value" "SYM_Arrow_XLarge" (at 150.622 146.05 0)
-      (effects (font (size 1 1)) hide)
+      (effects (font (size 1.27 1.27)) hide)
     )
     (property "Footprint" "" (at 148.59 146.05 0)
-      (effects (font (size 1 1)) hide)
+      (effects (font (size 1.27 1.27)) hide)
     )
     (property "Datasheet" "~" (at 148.59 146.05 0)
-      (effects (font (size 1 1)) hide)
+      (effects (font (size 1.27 1.27)) hide)
     )
     (property "Sim.Enable" "0" (at 148.59 146.05 0)
-      (effects (font (size 1 1)) hide)
+      (effects (font (size 1.27 1.27)) hide)
     )
     (instances
@@
     (in_bom no) (on_board no) (dnp no) (fields_autoplaced)
     (property "Reference" "#SYM7" (at 138.176 152.4 0)
-      (effects (font (size 1 1)) hide)
+      (effects (font (size 1.27 1.27)) hide)
     )
     (property "Value" "SYM_Arrow_XLarge" (at 133.858 152.4 0)
-      (effects (font (size 1 1)) hide)
+      (effects (font (size 1.27 1.27)) hide)
     )
     (property "Footprint" "" (at 135.89 152.4 0)
-      (effects (font (size 1 1)) hide)
+      (effects (font (size 1.27 1.27)) hide)
     )
     (property "Datasheet" "~" (at 135.89 152.4 0)
-      (effects (font (size 1 1)) hide)
+      (effects (font (size 1.27 1.27)) hide)
     )
     (property "Sim.Enable" "0" (at 135.89 152.4 0)
-      (effects (font (size 1 1)) hide)
+      (effects (font (size 1.27 1.27)) hide)
     )
     (instances
@@
     (in_bom no) (on_board no) (dnp no)
     (property "Reference" "#SYM5" (at 182.88 115.824 0)
-      (effects (font (size 1 1)) hide)
+      (effects (font (size 1.27 1.27)) hide)
     )
     (property "Value" "SYM_Arrow_XLarge" (at 182.88 120.142 0)
-      (effects (font (size 1 1)) hide)
+      (effects (font (size 1.27 1.27)) hide)
     )
     (property "Footprint" "" (at 182.88 118.11 0)
-      (effects (font (size 1 1)) hide)
+      (effects (font (size 1.27 1.27)) hide)
     )
     (property "Datasheet" "~" (at 182.88 118.11 0)
-      (effects (font (size 1 1)) hide)
+      (effects (font (size 1.27 1.27)) hide)
     )
     (property "Sim.Enable" "0" (at 182.88 118.11 0)
-      (effects (font (size 1 1)) hide)
+      (effects (font (size 1.27 1.27)) hide)
     )
     (instances
@@
     )
   )
-  (sheet (at 360.68 231.14) (size 276.86 189.23) (fields_autoplaced)
-    (stroke (width 0.1524) (type solid))
-    (fill (color 0 0 0 0.0000))
-    (property "Sheetname" "MSP430FR5994" (at 360.68 230.4284 0)
-      (effects (font (size 1 1)) (justify left bottom))
-    )
-    (property "Sheetfile" "MSP430FR5994.kicad_sch" (at 360.68 420.9546 0)
-      (effects (font (size 1 1)) (justify left top))
-    )
-    (instances
-      (project "LiFi_Receiver"
-        (path "/00b0bd1a-ca4b-4e13-a567-185f08cebf70" (page "6"))
-      )
-    )
-  )
   (sheet (at 13.97 -234.95) (size 276.86 187.96) (fields_autoplaced)
     (stroke (width 0.1524) (type solid))
     (fill (color 0 0 0 0.0000))
     (property "Sheetname" "RF_Backscatter" (at 13.97 -235.6616 0)
-      (effects (font (size 1 1)) (justify left bottom))
+      (effects (font (size 1.27 1.27)) (justify left bottom))
     )
     (property "Sheetfile" "RF_Backscatter.kicad_sch" (at 13.97 -46.4054 0)
-      (effects (font (size 1 1)) (justify left top))
+      (effects (font (size 1.27 1.27)) (justify left top))
     )
     (instances
@@
     (fill (color 0 0 0 0.0000))
     (property "Sheetname" "RHT Sensors" (at -346.71 10.7184 0)
-      (effects (font (size 1 1)) (justify left bottom))
+      (effects (font (size 1.27 1.27)) (justify left bottom))
     )
     (property "Sheetfile" "RHT_Sensors.kicad_sch" (at -346.71 201.2446 0)
-      (effects (font (size 1 1)) (justify left top))
+      (effects (font (size 1.27 1.27)) (justify left top))
     )
     (instances
@@
     (fill (color 0 0 0 0.0000))
     (property "Sheetname" "LiFi_Receiver_and_Power" (at 358.14 10.7184 0)
-      (effects (font (size 1 1)) (justify left bottom))
+      (effects (font (size 1.27 1.27)) (justify left bottom))
     )
     (property "Sheetfile" "ReceiverAndPower.kicad_sch" (at 358.14 199.9746 0)
-      (effects (font (size 1 1)) (justify left top))
+      (effects (font (size 1.27 1.27)) (justify left top))
     )
     (instances
@@
     (fill (color 0 0 0 0.0000))
     (property "Sheetname" "Peripherals" (at 12.7 230.4284 0)
-      (effects (font (size 1 1)) (justify left bottom))
+      (effects (font (size 1.27 1.27)) (justify left bottom))
     )
     (property "Sheetfile" "Peripherals.kicad_sch" (at 12.7 420.9546 0)
-      (effects (font (size 1 1)) (justify left top))
-    )
-    (instances
+      (effects (font (size 1.27 1.27)) (justify left top))
+    )
+    (instances
