File: PassiveLiFiTag/LiFi_Receiver/LiFi_Receiver.kicad_pcb (KiCad board)
At the start: 2 copper layers, 5 parts

Commit message: added updates
Parts:
- added J2: Conn_01x02, Connector_PinSocket_2.54mm:PinSocket_1x02_P2.54mm_Vertical, F.Cu at (156.4, 73.7)
- added J3: Conn_01x02, Connector_PinSocket_2.54mm:PinSocket_1x02_P2.54mm_Vertical, F.Cu at (161.0, 73.7)
- added J4: Conn_01x02, Connector_PinSocket_2.54mm:PinSocket_1x02_P2.54mm_Vertical, F.Cu at (165.6, 73.7)
- added J5: Conn_01x02, Connector_PinSocket_2.54mm:PinSocket_1x02_P2.54mm_Vertical, F.Cu at (170.2, 73.7)
- added U10: ADG721BRMZ-REEL, LIFI-FOOTPRINTS:RM_8_ADI-M, F.Cu at (106.7, 114.3)
- added U6: ADG722BRMZ-REEL7, LIFI-FOOTPRINTS:RM_8_ADI-M, F.Cu at (121.9, 86.7)
- added U7: ADG722BRMZ-REEL7, LIFI-FOOTPRINTS:RM_8_ADI-M, F.Cu at (99.1, 88.9)
- added U8: ADG721BRMZ-REEL, LIFI-FOOTPRINTS:RM_8_ADI-M, F.Cu at (111.8, 96.5)
- added U9: ADG721BRMZ-REEL, LIFI-FOOTPRINTS:RM_8_ADI-M, F.Cu at (121.9, 112.3)
- moved C15 40.2 mm to (111.8, 100.7), turned to 180 degrees
Routing:
- net Batt_ok: track 0.00 -> 23.6 mm

Commit message: Added updates
Parts:
- moved C16 77.7 mm to (141.2, 84.9)
- moved C17 77.0 mm to (131.0, 92.5)
- moved C14 68.7 mm to (141.1, 77.4)
- moved C13 51.2 mm to (131.0, 77.5)
- moved U7 44.6 mm to (141.3, 74.4)
- moved U9 36.3 mm to (141.3, 81.7)
- moved U10 35.1 mm to (131.3, 89.3)
- moved J2 26.6 mm to (131.8, 63.4)
- moved J3 26.2 mm to (136.8, 63.4)
- moved J4 25.9 mm to (141.8, 63.4)
- moved J5 25.5 mm to (146.8, 63.4)
- moved C15 25.0 mm to (131.1, 84.7)
- moved U8 24.5 mm to (131.3, 81.7)
- moved U6 15.5 mm to (131.3, 74.4)
Routing:
- net P3+: track 0.00 -> 64.3 mm, vias 0 -> 2
- net Batt_ok: track 23.6 -> 85.9 mm, vias 0 -> 10
- net VCC: track 0.00 -> 61.9 mm, vias 0 -> 4
- net P3-: track 0.00 -> 60.0 mm, vias 0 -> 3
- net P2-: track 0.00 -> 58.2 mm, vias 0 -> 5
- net P1-: track 0.00 -> 44.8 mm, vias 0 -> 4
- net P2+: track 0.00 -> 38.8 mm, vias 0 -> 3
- net P4-: track 0.00 -> 34.4 mm, vias 0 -> 1
- net P4+: track 0.00 -> 29.1 mm, vias 0 -> 4
- net P1+: track 0.00 -> 24.7 mm
- net GND: track 0.00 -> 3.16 mm, vias 0 -> 2
- added copper zone on B.Cu, net GND
- added copper zone on F.Cu, net GND
Other:
- board text added: "+"
- board text added: "-"
- board text added: "PV Array Input"
- board text added: "PV Array Switching Circuit"

Commit message: added updates
Parts:
- added C11: .1uF, Capacitor_SMD:C_01005_0402Metric, F.Cu at (137.9, 128.2)
- added C12: .1uF, Capacitor_SMD:C_01005_0402Metric, F.Cu at (148.8, 128.2)
- added RN1: 742C083472JP, LIFI-FOOTPRINTS:Res_network, F.Cu at (142.9, 117.6)
- added U4: HDC2080DMBR, LIFI-FOOTPRINTS:HDC2080_1, F.Cu at (134.8, 127.7)
- added U5: HDC2080DMBR, LIFI-FOOTPRINTS:HDC2080_1, F.Cu at (145.8, 127.6)
Routing:
- net GND: track 3.16 -> 32.7 mm, vias 2 -> 5
- net Net-(U5-SDA): track 0.00 -> 18.7 mm
- net Net-(U5-SCL): track 0.00 -> 18.7 mm
- net Net-(U4-SDA): track 0.00 -> 15.4 mm
- net Net-(U4-SCL): track 0.00 -> 13.4 mm
- net VCC: track 61.9 -> 74.5 mm
Other:
- board outline added: 21.9 x 11.8 mm
- board text added: "ADD FUSION SLOTS"
- board text added: "RH/T Sensors"

Commit message: added updates
Parts:
- added C10: 1n, Capacitor_SMD:C_01005_0402Metric, F.Cu at (197.7, 113.3)
- added R4: 27K, Resistor_SMD:R_01005_0402Metric, F.Cu at (197.7, 115.0)
- added SW1: SW_Push, LIFI-FOOTPRINTS:SW_TL59NF160Q, F.Cu at (192.6, 105.8)
Changed lines of the file:
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@@
   (net 19 "Net-(U4-SCL)")
   (net 20 "Net-(U5-SDA)")
+  (net 21 "~{RST}{slash}SBWTDIO_N")
+  (footprint "Capacitor_SMD:C_01005_0402Metric" (layer "F.Cu")
+    (at 197.725 113.325)
+    (descr "Capacitor SMD 01005 (0402 Metric), square (rectangular) end terminal, IPC_7351 nominal, (Body size source: http://www.vishay.com/docs/20056/crcw01005e3.pdf), generated with kicad-footprint-generator")
+    (tags "capacitor")
+    (property "Sheetfile" "Peripherals.kicad_sch")
+    (property "Sheetname" "Peripherals")
+    (property "ki_description" "Unpolarized capacitor, small symbol")
+    (property "ki_keywords" "capacitor cap")
+    (attr smd)
+    (fp_text reference "C10" (at 0 -1) (layer "F.SilkS")
+        (effects (font (size 1 1) (thickness 0.15)))
+    )
+    (fp_text value "1n" (at 0 1) (layer "F.Fab")
+        (effects (font (size 1 1) (thickness 0.15)))
+    )
+    (fp_text user "${REFERENCE}" (at 0 -0.62) (layer "F.Fab")
+        (effects (font (size 0.25 0.25) (thickness 0.04)))
+    )
+    (fp_line (start -0.6 -0.3) (end 0.6 -0.3)
+      (stroke (width 0.05) (type solid)) (layer "F.CrtYd"))
+    (fp_line (start -0.6 0.3) (end -0.6 -0.3)
+      (stroke (width 0.05) (type solid)) (layer "F.CrtYd"))
+    (fp_line (start 0.6 -0.3) (end 0.6 0.3)
+      (stroke (width 0.05) (type solid)) (layer "F.CrtYd"))
+    (fp_line (start 0.6 0.3) (end -0.6 0.3)
+      (stroke (width 0.05) (type solid)) (layer "F.CrtYd"))
+    (fp_line (start -0.2 -0.1) (end 0.2 -0.1)
+      (stroke (width 0.1) (type solid)) (layer "F.Fab"))
+    (fp_line (start -0.2 0.1) (end -0.2 -0.1)
+      (stroke (width 0.1) (type solid)) (layer "F.Fab"))
+    (fp_line (start 0.2 -0.1) (end 0.2 0.1)
+      (stroke (width 0.1) (type solid)) (layer "F.Fab"))
+    (fp_line (start 0.2 0.1) (end -0.2 0.1)
+      (stroke (width 0.1) (type solid)) (layer "F.Fab"))
+    (pad "" smd roundrect (at -0.275 0) (size 0.27 0.27) (layers "F.Paste") (roundrect_rratio 0.25))
+    (pad "" smd roundrect (at 0.275 0) (size 0.27 0.27) (layers "F.Paste") (roundrect_rratio 0.25))
+    (pad "1" smd roundrect (at -0.25 0) (size 0.4 0.3) (layers "F.Cu" "F.Mask") (roundrect_rratio 0.25)
+      (net 21 "~{RST}{slash}SBWTDIO_N") (pintype "passive"))
+    (pad "2" smd roundrect (at 0.25 0) (size 0.4 0.3) (layers "F.Cu" "F.Mask") (roundrect_rratio 0.25)
+      (net 2 "GND") (pintype "passive"))
+    (model "${KICAD6_3DMODEL_DIR}/Capacitor_SMD.3dshapes/C_01005_0402Metric.wrl"
+      (offset (xyz 0 0 0))
+      (scale (xyz 1 1 1))
+      (rotate (xyz 0 0 0))
+    )
+  )
   (footprint "Capacitor_SMD:C_01005_0402Metric" (layer "F.Cu")
     (at 148.825 128.150001 -90)
@@
       (net 1 "VCC") (pinfunction "VDD") (pintype "power_in"))
   )
+  (footprint "LIFI-FOOTPRINTS:SW_TL59NF160Q" (layer "F.Cu")
+    (at 192.575 105.85)
+    (property "Sheetfile" "Peripherals.kicad_sch")
+    (property "Sheetname" "Peripherals")
+    (property "ki_description" "Push button switch, generic, two pins")
+    (property "ki_keywords" "switch normally-open pushbutton push-button")
+    (attr through_hole)
+    (fp_text reference "SW1" (at -0.369 -4.985) (layer "F.SilkS")
+        (effects (font (size 1 1) (thickness 0.15)))
+    )
+    (fp_text value "SW_Push" (at 4.711 4.985) (layer "F.Fab")
+        (effects (font (size 1 1) (thickness 0.15)))
+    )
+    (fp_line (start -3.1 -2.9) (end 3.1 -2.9)
+      (stroke (width 0.127) (type solid)) (layer "F.SilkS"))
+    (fp_line (start -3.1 -1.074) (end -3.1 -2.9)
+      (stroke (width 0.127) (type solid)) (layer "F.SilkS"))
+    (fp_line (start -3.1 3.3) (end -3.1 1.074)
+      (stroke (width 0.127) (type solid)) (layer "F.SilkS"))
+    (fp_line (start 3.1 -2.9) (end 3.1 -1.074)
+      (stroke (width 0.127) (type solid)) (layer "F.SilkS"))
+    (fp_line (start 3.1 3.3) (end -3.1 3.3)
+      (stroke (width 0.127) (type solid)) (layer "F.SilkS"))
+    (fp_line (start 3.1 3.3) (end 3.1 1.074)
+      (stroke (width 0.127) (type solid)) (layer "F.SilkS"))
+    (fp_circle (center -4.294 0) (end -4.194 0)
+      (stroke (width 0.2) (type solid)) (fill none) (layer "F.SilkS"))
+    (fp_line (start -3.544 -3.15) (end -3.544 3.55)
+      (stroke (width 0.05) (type solid)) (layer "F.CrtYd"))
+    (fp_line (start -3.544 3.55) (end 3.544 3.55)
+      (stroke (width 0.05) (type solid)) (layer "F.CrtYd"))
+    (fp_line (start 3.544 -3.15) (end -3.544 -3.15)
+      (stroke (width 0.05) (type solid)) (layer "F.CrtYd"))
+    (fp_line (start 3.544 3.55) (end 3.544 -3.15)
+      (stroke (width 0.05) (type solid)) (layer "F.CrtYd"))
+    (fp_line (start -3.1 -2.9) (end 3.1 -2.9)
+      (stroke (width 0.127) (type solid)) (layer "F.Fab"))
+    (fp_line (start -3.1 3.3) (end -3.1 -2.9)
+      (stroke (width 0.127) (type solid)) (layer "F.Fab"))
+    (fp_line (start 3.1 -2.9) (end 3.1 3.3)
+      (stroke (width 0.127) (type solid)) (layer "F.Fab"))
+    (fp_line (start 3.1 3.3) (end -3.1 3.3)
+      (stroke (width 0.127) (type solid)) (layer "F.Fab"))
+    (fp_circle (center -4.294 0) (end -4.194 0)
+      (stroke (width 0.2) (type solid)) (fill none) (layer "F.Fab"))
+    (pad "1" thru_hole rect (at -2.5 0) (size 1.508 1.508) (drill 1) (layers "*.Cu" "*.Mask")
+      (net 2 "GND") (pinfunction "1") (pintype "passive") (solder_mask_margin 0.102))
+    (pad "2" thru_hole circle (at 2.5 0) (size 1.508 1.508) (drill 1) (layers "*.Cu" "*.Mask")
+      (net 21 "~{RST}{slash}SBWTDIO_N") (pinfunction "2") (pintype "passive") (solder_mask_margin 0.102))
+  )
   (footprint "Capacitor_SMD:C_01005_0402Metric" (layer "F.Cu")
     (at 131.0863 84.7273 180)
@@
       (offset (xyz 0 0 0))
       (scale (xyz 1 1 1))
+      (rotate (xyz 0 0 0))
+    )
+  )
+  (footprint "Resistor_SMD:R_01005_0402Metric" (layer "F.Cu")
+    (at 197.725 114.975)
+    (descr "Resistor SMD 01005 (0402 Metric), square (rectangular) end terminal, IPC_7351 nominal, (Body size source: http://www.vishay.com/docs/20056/crcw01005e3.pdf), generated with kicad-footprint-generator")
+    (tags "resistor")
+    (property "Sheetfile" "Peripherals.kicad_sch")
+    (property "Sheetname" "Peripherals")
+    (property "ki_description" "Resistor, small US symbol")
+    (property "ki_keywords" "r resistor")
+    (attr smd)
+    (fp_text reference "R4" (at 0 -1) (layer "F.SilkS")
+        (effects (font (size 1 1) (thickness 0.15)))
+    )
+    (fp_text value "27K" (at 0 1) (layer "F.Fab")
+        (effects (font (size 1 1) (thickness 0.15)))
+    )
+    (fp_text user "${REFERENCE}" (at 0 -0.62) (layer "F.Fab")
+        (effects (font (size 0.25 0.25) (thickness 0.04)))
+    )
+    (fp_line (start -0.6 -0.3) (end 0.6 -0.3)
+      (stroke (width 0.05) (type solid)) (layer "F.CrtYd"))
+    (fp_line (start -0.6 0.3) (end -0.6 -0.3)
+      (stroke (width 0.05) (type solid)) (layer "F.CrtYd"))
+    (fp_line (start 0.6 -0.3) (end 0.6 0.3)
+      (stroke (width 0.05) (type solid)) (layer "F.CrtYd"))
+    (fp_line (start 0.6 0.3) (end -0.6 0.3)
+      (stroke (width 0.05) (type solid)) (layer "F.CrtYd"))
+    (fp_line (start -0.2 -0.1) (end 0.2 -0.1)
+      (stroke (width 0.1) (type solid)) (layer "F.Fab"))
+    (fp_line (start -0.2 0.1) (end -0.2 -0.1)
+      (stroke (width 0.1) (type solid)) (layer "F.Fab"))
+    (fp_line (start 0.2 -0.1) (end 0.2 0.1)
+      (stroke (width 0.1) (type solid)) (layer "F.Fab"))
+    (fp_line (start 0.2 0.1) (end -0.2 0.1)
+      (stroke (width 0.1) (type solid)) (layer "F.Fab"))
+    (pad "" smd roundrect (at -0.275 0) (size 0.27 0.27) (layers "F.Paste") (roundrect_rratio 0.25))
+    (pad "" smd roundrect (at 0.275 0) (size 0.27 0.27) (layers "F.Paste") (roundrect_rratio 0.25))
+    (pad "1" smd roundrect (at -0.25 0) (size 0.4 0.3) (layers "F.Cu" "F.Mask") (roundrect_rratio 0.25)
+      (net 1 "VCC") (pintype "passive"))
+    (pad "2" smd roundrect (at 0.25 0) (size 0.4 0.3) (layers "F.Cu" "F.Mask") (roundrect_rratio 0.25)
+      (net 21 "~{RST}{slash}SBWTDIO_N") (pintype "passive"))
+    (model "${KICAD6_3DMODEL_DIR}/Resistor_SMD.3dshapes/R_01005_0402Metric.wrl"
+      (offset (xyz 0 0 0))
+      (scale (xyz 1 1 1))

Commit message: Added updates
Parts:
- added C1: 100n, Capacitor_SMD:C_01005_0402Metric, F.Cu at (222.1, 70.8)
- added C2: 100n, Capacitor_SMD:C_01005_0402Metric, F.Cu at (235.6, 74.0)
- added C3: 100n, Capacitor_SMD:C_01005_0402Metric, F.Cu at (235.6, 75.6)
- added C4: 100n, Capacitor_SMD:C_01005_0402Metric, F.Cu at (235.6, 77.3)
- added C5: 10u, Capacitor_SMD:C_01005_0402Metric, F.Cu at (235.6, 78.9)
- added C6: 22p, Capacitor_SMD:C_01005_0402Metric, F.Cu at (235.6, 80.6)
- added C7: 22p, Capacitor_SMD:C_01005_0402Metric, F.Cu at (235.6, 82.2)
- added J1: Conn_01x07, Connector_PinSocket_2.54mm:PinSocket_1x07_P2.54mm_Vertical, F.Cu at (84.2, 72.6)
- added R1: 0R, Resistor_SMD:R_01005_0402Metric, F.Cu at (230.9, 88.7)
- added U1: MSP430FR5994IPNR, Library:PN0080A_L, F.Cu at (226.6, 79.4)
- added Y1: Crystal_Small, Library:xtal-2, F.Cu at (240.6, 81.2)
- moved R4 106.3 mm to (92.3, 129.2)
- moved C10 103.0 mm to (95.9, 129.2)
- moved SW1 100.3 mm to (94.1, 124.9)
- moved RN1 0.18 mm to (143.1, 117.6)
Routing:
- net VCC: track 74.5 -> 89.0 mm, vias 4 -> 6
- net GND: track 32.7 -> 45.5 mm, vias 5 -> 7
- net ~{RST}/SBWTDIO_N: track 0.00 -> 7.79 mm
- net Net-(U5-SDA): track 18.7 -> 15.3 mm
- net Net-(U5-SCL): track 18.7 -> 15.8 mm
Other:
- board outline removed
- board text added: "**ADD FUSION SLOTS**"
- board text added: "EZFET/JTAG"
- board text added: "Gnd 3.3V RXD TXD RST/SBWTDIO TEST_SBWTCK"
- board text added: "RST"
- board text removed: "ADD FUSION SLOTS"

Commit message: Added Updates
Parts:
- moved C5 24.4 mm to (212.7, 70.5), turned to 90 degrees
- moved Y1 23.9 mm to (221.1, 67.2)
- moved C6 22.7 mm to (219.9, 64.2), turned to -90 degrees
- moved C7 22.4 mm to (222.3, 64.2), turned to -90 degrees
- moved R1 22.4 mm to (215.1, 72.9)
- moved C4 19.8 mm to (217.9, 86.1), turned to 90 degrees
- moved C3 12.2 mm to (233.4, 87.6), turned to 180 degrees
- moved C1 5.28 mm to (217.3, 73.2), turned to -90 degrees
- moved C2 1.35 mm to (235.0, 72.8)
Routing:
- net GND: track 45.5 -> 66.8 mm, vias 7 -> 8
- net VCC: track 89.0 -> 100.1 mm
- net Net-(U1-PJ.5_LFXOUT): track 0.00 -> 9.53 mm
- net Net-(U1-PJ.4_LFXIN): track 0.00 -> 8.73 mm
- net AVCC_DVSS_: track 0.00 -> 6.56 mm

Commit message: Added Updates
Parts:
- C5: footprint Capacitor_SMD:C_01005_0402Metric -> LIFI-FOOTPRINTS:TAJA_AVX-M
- moved J1 105.9 mm to (188.2, 92.6)
- moved C5 98.8 mm to (115.1, 85.7)
- moved C3 96.9 mm to (138.0, 104.7)
- moved C6 96.9 mm to (124.5, 81.3)
- moved C7 96.9 mm to (126.9, 81.3)
- moved R1 96.9 mm to (119.7, 90.0)
- moved U1 96.9 mm to (131.2, 96.5)
- moved Y1 96.9 mm to (125.7, 84.3)
- moved C1 96.9 mm to (121.9, 90.3)
- moved C2 96.9 mm to (139.6, 89.9)
- moved C4 96.9 mm to (122.4, 103.2)
- moved R4 71.5 mm to (163.8, 132.3)
- moved C10 71.5 mm to (167.3, 132.3)
- moved SW1 71.5 mm to (165.5, 128.0)
- moved C16 61.8 mm to (83.3, 106.5)
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Routing:
- net GND: track 66.8 -> 52.0 mm
- net VCC: track 100.1 -> 105.6 mm
Other:
- board text added: "MSP430FR994"

Commit message: Added updates
Parts:
- added C8: C_Small, Capacitor_SMD:C_0402_1005Metric, F.Cu at (73.8, 65.0)
- added C9: C_Small, Capacitor_SMD:C_0402_1005Metric, F.Cu at (109.5, 57.5)
- added R2: R_Small_US, Resistor_SMD:R_0402_1005Metric, F.Cu at (76.2, 65.5)
- added R3: R_Small_US, Resistor_SMD:R_0402_1005Metric, F.Cu at (107.1, 57.0)
- added U2: TS881ILT, LIFI-FOOTPRINTS:TS88_3, F.Cu at (80.4, 64.0)
Connections:
- C1 pad 2: GND -> P4-
- C10 pad 2: GND -> P4-
- C11 pad 2: GND -> P4-
- C12 pad 2: GND -> P4-
- C13 pad 2: GND -> P4-
- C14 pad 2: GND -> P4-
- C15 pad 2: GND -> P4-
- C16 pad 2: GND -> P4-
- C17 pad 2: GND -> P4-
- C2 pad 2: GND -> P4-
- C3 pad 2: GND -> P4-
- C4 pad 2: GND -> P4-
- C5 pad 2: GND -> P4-
- C6 pad 1: GND -> P4-
- C7 pad 1: GND -> P4-
- J1 pad 1: GND -> P4-
- SW1 pad 1: GND -> P4-
- U1 pad 19: GND -> P4-
- U1 pad 39: GND -> P4-
- U1 pad 60: GND -> P4-
- U1 pad 73: GND -> P4-
- U1 pad 76: GND -> P4-
- U1 pad 79: GND -> P4-
- U10 pad 4: GND -> P4-
- U4 pad 2: GND -> P4-
- U4 pad 4: GND -> P4-
- U5 pad 2: GND -> P4-
- U5 pad 3: GND -> P4-
- U5 pad 4: GND -> P4-
- U6 pad 4: GND -> P4-
- U7 pad 4: GND -> P4-
- U8 pad 4: GND -> P4-
- U9 pad 4: GND -> P4-
Routing:
- net GND: track 52.0 -> 0.00 mm, vias 8 -> 0
- net P4-: track 34.4 -> 86.5 mm, vias 1 -> 9
- net Net-(U2-IN+): track 0.00 -> 4.84 mm
- net Harvester_In: track 0.00 -> 1.90 mm
- added copper zone on B.Cu, net P4-
- added copper zone on F.Cu, net P4-
- removed copper zone on B.Cu, net GND
- removed copper zone on F.Cu, net GND
Other:
- board text added: "1b ADC"
