File: PassiveLiFiTag/LiFi_Receiver/LiFi_Receiver.kicad_pcb (KiCad board)
At the start: 2 copper layers, 38 parts, among them J1 Conn_01x07, J2 Conn_01x02, J3 Conn_01x02, J4 Conn_01x02, J5 Conn_01x02, SW1 SW_Push, U1 MSP430FR5994IPNR, U10 ADG721BRMZ-REEL, U2 TS881ILT, U4 HDC2080DMBR, U5 HDC2080DMBR, U6 ADG722BRMZ-REEL7, U7 ADG722BRMZ-REEL7, U8 ADG721BRMZ-REEL, U9 ADG721BRMZ-REEL, Y1 Crystal_Small

Commit message: Added Updates
Parts:
- added JP1: SolderJumper_2_Open, Jumper:SolderJumper-2_P1.3mm_Open_TrianglePad1.0x1.5mm, F.Cu at (129.5, 133.2)
- added JP2: SolderJumper_2_Open, Jumper:SolderJumper-2_P1.3mm_Open_TrianglePad1.0x1.5mm, F.Cu at (135.0, 133.2)
- added JP3: SolderJumper_2_Open, Jumper:SolderJumper-2_P1.3mm_Open_TrianglePad1.0x1.5mm, F.Cu at (138.6, 146.8)
- moved RN1 9.71 mm to (136.8, 139.8)
- moved C12 0.47 mm to (133.2, 150.3)
- moved U5 0.47 mm to (130.2, 149.8)
- moved C11 0.47 mm to (122.3, 150.4)
- moved U4 0.47 mm to (119.2, 149.9)
Connections:
- C12 pad 1: VCC -> Net-(JP3-B)
- RN1 pad 5: scl1 -> Net-(JP1-B)
- U5 pad 5: VCC -> Net-(JP3-B)
Routing:
- net Net-(U5-SCL): track 15.8 -> 30.7 mm, vias 0 -> 2
- net Net-(JP1-B): track 0.00 -> 13.5 mm, vias 0 -> 2
- net scl2: track 0.00 -> 11.3 mm, vias 0 -> 2
- net Net-(U5-SDA): track 15.3 -> 25.3 mm, vias 0 -> 2
- net Net-(JP3-B): track 0.00 -> 9.66 mm
- net Net-(U4-SCL): track 13.2 -> 22.6 mm
- net Net-(U4-SDA): track 15.4 -> 24.9 mm
- net VCC: track 105.6 -> 99.3 mm, vias 6 -> 5

Commit message: Added Updates
Parts:
- added C18: C_Small, Connector_PinSocket_2.54mm:PinSocket_1x02_P2.54mm_Vertical, F.Cu at (110.5, 82.8)
- added C19: C_Small, Connector_PinSocket_2.54mm:PinSocket_1x02_P2.54mm_Vertical, F.Cu at (144.2, 58.1)
- added C20: 4.7uF, Capacitor_SMD:C_01005_0402Metric, F.Cu at (123.0, 88.7)
- added C21: 0.1uF, Capacitor_SMD:C_01005_0402Metric, F.Cu at (123.0, 89.5)
- added C22: 22uF, Capacitor_SMD:C_01005_0402Metric, F.Cu at (131.9, 91.1)
- added C23: 0.01uF, Capacitor_SMD:C_01005_0402Metric, F.Cu at (123.5, 93.3)
- added C24: 4.7uF, Capacitor_SMD:C_01005_0402Metric, F.Cu at (123.5, 92.3)
- added C25: 0.1uF, Capacitor_SMD:C_01005_0402Metric, F.Cu at (142.5, 89.0)
- added C26: 0.1uF, Capacitor_SMD:C_01005_0402Metric, F.Cu at (148.6, 89.1)
- added JP5: Jumper_3_Open, Connector_PinHeader_2.54mm:PinHeader_1x03_P2.54mm_Vertical, F.Cu at (120.0, 77.6)
- added JP6: Jumper_3_Open, Connector_PinHeader_2.54mm:PinHeader_1x03_P2.54mm_Vertical, F.Cu at (138.8, 60.6)
- added L1: 22uH, Inductor_SMD:L_01005_0402Metric, F.Cu at (125.2, 88.3)
- added L2: 4.7uH, Inductor_SMD:L_01005_0402Metric, F.Cu at (130.5, 89.0)
- added R5: R_Small_US, Connector_PinSocket_2.54mm:PinSocket_1x02_P2.54mm_Vertical, F.Cu at (114.7, 85.3)
- added R6: R_Small_US, Connector_PinSocket_2.54mm:PinSocket_1x02_P2.54mm_Vertical, F.Cu at (148.3, 58.1)
- added U11: S-1313B24-M5T1U3, Package_TO_SOT_SMD:SOT-23-5, F.Cu at (145.5, 89.8)
- added U3: BQ25570RGRR, Library:Bat_Harv2, F.Cu at (127.4, 91.3)
- moved U2 66.8 mm to (146.3, 53.1)
- moved R2 64.0 mm to (138.9, 52.6)
- moved C8 64.0 mm to (136.5, 52.1)
- moved C3 51.6 mm to (189.5, 101.1)
- moved C6 51.6 mm to (176.0, 77.6)
- moved C7 51.6 mm to (178.4, 77.6)
- moved R1 51.6 mm to (171.1, 86.4)
- moved Y1 51.6 mm to (177.2, 80.7)
- moved C1 51.6 mm to (173.3, 86.6)
- moved C2 51.6 mm to (191.0, 86.2)
- moved C4 51.6 mm to (173.9, 99.6)
- moved C5 51.6 mm to (166.6, 82.1)
- moved U1 51.6 mm to (182.6, 92.9)
- moved C10 44.6 mm to (210.9, 123.0)
- moved SW1 44.6 mm to (209.1, 118.6)
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Connections:
- net Harvester_In renamed Net-(JP5-A)
- net P4- renamed GND
- C8 pad 2: Net-(U2-IN+) -> Net-(JP6-B)
- R2 pad 1: Net-(U2-IN+) -> Net-(JP6-B)
- U2 pad 3: Net-(U2-IN+) -> Comparator_In
Routing:
- net GND: track 86.5 -> 108.7 mm, vias 9 -> 14
- net VCC: track 99.3 -> 118.1 mm, vias 5 -> 6
- net Harvester_In: track 0.00 -> 17.1 mm, vias 0 -> 2
- net Comparator_In: track 0.00 -> 12.4 mm
- net Net-(JP6-B): track 0.00 -> 11.9 mm
- net Harvester_out: track 0.00 -> 10.5 mm
- net Net-(JP6-A): track 0.00 -> 10.5 mm
- net Net-(U3-VOC_SAMP): track 0.00 -> 10.2 mm, vias 0 -> 2
- net Net-(JP5-B): track 0.00 -> 9.61 mm
- net P1+: track 24.7 -> 33.9 mm, vias 0 -> 1
- net Net-(JP5-A): track 1.90 -> 7.98 mm
- net Net-(U2-IN+): track 4.84 -> 0.00 mm
- net Net-(U3-VREF_SAMP): track 0.00 -> 2.89 mm
- net Net-(U3-LBUCK): track 0.00 -> 2.05 mm
- net Net-(U3-LBOOST): track 0.00 -> 1.80 mm
Other:
- board outline added: 180.6 x 107.8 mm
- board text added: "2.4v Reg"
- board text added: "Battery Harvester/LPF"
- board text added: "Comparator/HPF"
- board text added: "SMD"
- board text added: "THT"
- board text removed: "**ADD FUSION SLOTS**"
- board text removed: "1b ADC"

Commit message: Design almost completed
Parts:
- removed SW1: SW_Push, LIFI-FOOTPRINTS:SW_TL59NF160Q
- added C27: DNP, Capacitor_SMD:C_0603_1608Metric, F.Cu at (138.4, 45.5)
- added C28: DNP, Capacitor_SMD:C_0603_1608Metric, F.Cu at (142.3, 45.5)
- added H1: MountingHole, MountingHole:MountingHole_2.2mm_M2, F.Cu at (52.3, 39.5)
- added H2: MountingHole, MountingHole:MountingHole_2.2mm_M2, F.Cu at (90.2, 39.6)
- added J6: Conn_01x08, Connector_PinHeader_2.54mm:PinHeader_2x04_P2.54mm_Vertical, F.Cu at (166.5, 63.1)
- added J7: Conn_01x08, Connector_PinHeader_2.54mm:PinHeader_2x04_P2.54mm_Vertical, F.Cu at (166.5, 76.2)
- added J9: Conn_01x02, Connector_PinSocket_2.54mm:PinSocket_1x02_P2.54mm_Vertical, F.Cu at (102.5, 103.8)
- added R10: R_Small_US, Resistor_SMD:R_0603_1608Metric, F.Cu at (92.3, 100.6)
- added R11: R_Small_US, Resistor_SMD:R_0603_1608Metric, F.Cu at (87.3, 100.6)
- added R12: R_Small_US, Resistor_SMD:R_0603_1608Metric, F.Cu at (82.3, 100.6)
- added R13: R_Small_US, Resistor_SMD:R_0603_1608Metric, F.Cu at (92.3, 96.6)
- added R7: R_Small_US, Resistor_SMD:R_0603_1608Metric, F.Cu at (92.3, 104.6)
- added R8: R_Small_US, Resistor_SMD:R_0603_1608Metric, F.Cu at (87.3, 104.6)
- added R9: R_Small_US, Resistor_SMD:R_0603_1608Metric, F.Cu at (82.3, 104.6)
- added SW2: PTS645SL43SMTR92LFS, Library:PTS645SL43SMTR92LFS_CNK-M, F.Cu at (98.9, 51.9)
- added TP1: TestPoint, TestPoint:TestPoint_Pad_D1.5mm, F.Cu at (102.3, 99.1)
- added TP2: TestPoint, TestPoint:TestPoint_Pad_D1.5mm, F.Cu at (105.1, 99.1)
- added TP3: SDA, TestPoint:TestPoint_Pad_D1.5mm, F.Cu at (118.6, 84.4)
- added TP4: SCL, TestPoint:TestPoint_Pad_D1.5mm, F.Cu at (126.2, 83.5)
- added TP5: 2.4v, TestPoint:TestPoint_Pad_D1.5mm, F.Cu at (112.7, 88.7)
- added Y2: Crystal_Small, Library:xtal-2, F.Cu at (140.3, 42.6)
- C1, C10, C11, C12, C13, C14, C15, C16, C17, C2, C20, C21, C22, C23, C24, C25, C26, C3, C4, C6, C7: footprint Capacitor_SMD:C_01005_0402Metric -> Capacitor_SMD:C_0603_1608Metric
- C5: footprint LIFI-FOOTPRINTS:TAJA_AVX-M -> Capacitor_SMD:C_0603_1608Metric
- C8, C9: footprint Capacitor_SMD:C_0402_1005Metric -> Capacitor_SMD:C_0603_1608Metric
- L1, L2: footprint Inductor_SMD:L_01005_0402Metric -> Inductor_SMD:L_0603_1608Metric
- R1, R4: footprint Resistor_SMD:R_01005_0402Metric -> Resistor_SMD:R_0603_1608Metric
- R2, R3: footprint Resistor_SMD:R_0402_1005Metric -> Resistor_SMD:R_0603_1608Metric
- RN1: footprint LIFI-FOOTPRINTS:Res_network -> Library:RESCAV80P320X160X70-8N
- U10, U8, U9: footprint LIFI-FOOTPRINTS:RM_8_ADI-M -> Library:RM_8_ADI
- U2: footprint LIFI-FOOTPRINTS:TS88_3 -> Library:SOT23-5_TS881_TEX
- U3: footprint Library:Bat_Harv2 -> Library:Bat_Harv1
- U4, U5: footprint LIFI-FOOTPRINTS:HDC2080_1 -> Library:DMB0006A_NV
- U6, U7: footprint LIFI-FOOTPRINTS:RM_8_ADI-M -> Library:RM_8_ADI-M
- moved R4 127.6 mm to (96.8, 59.2)
- moved C10 127.2 mm to (100.9, 59.2)
- moved C3 81.7 mm to (119.1, 59.6), turned to 0 degrees
- moved C2 77.3 mm to (119.1, 57.7)
- moved J1 71.3 mm to (168.9, 41.9)
- moved C4 66.7 mm to (119.1, 61.5), turned to 0 degrees
- moved Y1 66.5 mm to (122.5, 42.8)
- moved C6 64.1 mm to (120.5, 45.5), turned to 0 degrees
- moved C7 62.7 mm to (124.5, 45.6), turned to 180 degrees
- moved C1 62.3 mm to (119.1, 55.9), turned to 0 degrees
- moved JP5 58.8 mm to (64.0, 95.2), turned to 180 degrees
- moved R5 58.7 mm to (56.0, 87.6), turned to 0 degrees
- moved U1 57.8 mm to (131.4, 66.2)
- moved C9 57.7 mm to (59.5, 96.9), turned to 180 degrees
- moved R1 55.5 mm to (124.7, 55.9)
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Connections:
- J1 pad 3: +3.3V -> VCC
- JP1 pad 1: sda2 -> UCB2SDA_BYP
- JP1 pad 2: Net-(JP1-B) -> UCB2SDA
- JP2 pad 1: Net-(JP2-A) -> UCB2SCL_BYP
- JP2 pad 2: scl2 -> UCB2SCL
- RN1 pad 1: (no net) -> UCB2SDA
- RN1 pad 2: (no net) -> UCB2SCL
- RN1 pad 3: (no net) -> UCB2SDA_BYP
- RN1 pad 4: VCC -> UCB2SCL_BYP
- RN1 pad 5: Net-(JP1-B) -> VCC
- RN1 pad 6: (no net) -> VCC
- RN1 pad 7: (no net) -> VCC
- RN1 pad 8: (no net) -> VCC
- U1 pad 12: unconnected-(U1-P4.7-Pad12) -> Net-(J7-Pin_1)
- U1 pad 31: unconnected-(U1-P4.0_A8-Pad31) -> Net-(J7-Pin_8)
- U1 pad 32: unconnected-(U1-P4.1_A9-Pad32) -> Net-(J7-Pin_7)
- U1 pad 33: unconnected-(U1-P4.2_A10-Pad33) -> Net-(J7-Pin_6)
- U1 pad 34: unconnected-(U1-P4.3_A11-Pad34) -> Net-(J7-Pin_5)
- U1 pad 53: unconnected-(U1-P5.0_UCB1SIMO_UCB1SDA-Pad53) -> Net-(J6-Pin_1)
- U1 pad 54: unconnected-(U1-P5.1_UCB1SOMI_UCB1SCL-Pad54) -> Net-(J6-Pin_2)
- U1 pad 55: unconnected-(U1-P5.2_UCB1CLK_TA4CLK-Pad55) -> Net-(J6-Pin_3)
- U1 pad 56: unconnected-(U1-P5.3_UCB1STE-Pad56) -> Net-(J6-Pin_4)
- U1 pad 57: unconnected-(U1-P4.4_TB0.5-Pad57) -> Net-(J7-Pin_4)
- U1 pad 58: unconnected-(U1-P4.5-Pad58) -> Net-(J7-Pin_3)
- U1 pad 59: unconnected-(U1-P4.6-Pad59) -> Net-(J7-Pin_2)
- U1 pad 65: unconnected-(U1-P5.4_UCA2TXD_UCA2SIMO_TB0OUTH-Pad65) -> Net-(J6-Pin_5)
- U1 pad 66: unconnected-(U1-P5.5_UCA2RXD_UCA2SOMI_ACLK-Pad66) -> Net-(J6-Pin_6)
- U1 pad 67: unconnected-(U1-P5.6_UCA2CLK_TA4.0_SMCLK-Pad67) -> Net-(J6-Pin_7)
- U1 pad 68: unconnected-(U1-P5.7_UCA2STE_TA4.1_MCLK-Pad68) -> Net-(J6-Pin_8)
- U1 pad 74: unconnected-(U1-PJ.6_HFXIN-Pad74) -> Net-(U1-PJ.6_HFXIN)
- U1 pad 75: unconnected-(U1-PJ.7_HFXOUT-Pad75) -> Net-(U1-PJ.7_HFXOUT)
- U11 pad 4: (no net) -> unconnected-(U11-NC-Pad4)
- U3 pad 5: unconnected-(U3-EN_N-Pad5) -> GND
- U4 pad 1: Net-(U4-SDA) -> UCB2SDA
- U4 pad 6: Net-(U4-SCL) -> UCB2SCL
- U5 pad 1: Net-(U5-SDA) -> UCB2SDA_BYP
- U5 pad 6: Net-(U5-SCL) -> UCB2SCL_BYP
Routing:
- net VCC: track 118.1 -> 354.3 mm, vias 6 -> 13
- net P1+: track 33.9 -> 136.7 mm, vias 1 -> 2
- net ~{RST}/SBWTDIO_N: track 7.79 -> 105.5 mm, vias 0 -> 3
- net UCB2SCL: track 0.00 -> 70.1 mm, vias 0 -> 3
- net UCB2SDA: track 0.00 -> 69.5 mm, vias 0 -> 2
- net GND: track 108.7 -> 162.8 mm, vias 14 -> 28
- net TEST_SBWTCK: track 0.00 -> 53.0 mm, vias 0 -> 2
- net P2.0_UART_TXD: track 0.00 -> 52.1 mm, vias 0 -> 2
- net Net-(J7-Pin_2): track 0.00 -> 51.0 mm, vias 0 -> 2
- net Net-(J7-Pin_4): track 0.00 -> 46.7 mm, vias 0 -> 1
- net Net-(J6-Pin_8): track 0.00 -> 46.2 mm, vias 0 -> 2
- net Net-(J7-Pin_1): track 0.00 -> 45.8 mm, vias 0 -> 2
- net Net-(J7-Pin_8): track 0.00 -> 44.5 mm
- net Net-(J7-Pin_3): track 0.00 -> 43.8 mm, vias 0 -> 1
- net Net-(J6-Pin_6): track 0.00 -> 42.7 mm, vias 0 -> 2
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Other:
- board size 180.6 x 107.8 mm -> 132.6 x 80 mm
- board text added: "2.4V LinReg"
- board text added: "2.4v"
- board text added: "5vMax"
- board text added: "Bat In"
- board text added: "Bat+"
- board text added: "Bat-"
- board text added: "EZ-FET"
- board text added: "FR5994"
- board text added: "GND NC Vcc RXD TXD RST! TEST"
- board text added: "GPIO Extension"
- board text added: "Greener Greenhouses"
- board text added: "HF Oscillator"
- board text added: "HPF/1B ADC"
- board text added: "Harvester [BQ255]"
- board text added: "LF Oscillator"
- board text added: "LPF"
- board text added: "P4.6 P4.4 P4.2 P4.0"
- board text added: "P4.7 P4.5 P4.3 P4.1"
- board text added: "P5.0 P5.2 P5.4 P5.6"
- board text added: "P5.1 P5.3 P5.5 P5.7"
- board text added: "PV Input/MOSFET Config"
- board text added: "SCL"
- board text added: "SDA"
- board text added: "U3"
- board text added: "Y1"
- board text added: "Y2"
- board text added: "dnp"
- board text removed: "2.4v Reg"
- board text removed: "Battery Harvester/LPF"
- board text removed: "Comparator/HPF"
- board text removed: "EZFET/JTAG"
- board text removed: "Gnd 3.3V RXD TXD RST/SBWTDIO TEST_SBWTCK"
- board text removed: "MSP430FR994"
- board text removed: "PV Array Input"
- board text removed: "PV Array Switching Circuit"

Commit message: ready for design review
Parts:
- moved C23 4.60 mm to (79.7, 95.8), turned to 0 degrees
- moved C24 4.43 mm to (79.8, 97.5), turned to 0 degrees
- moved C6 0.63 mm to (119.9, 45.5)
- moved C7 0.63 mm to (123.8, 45.6)
- moved Y1 0.63 mm to (121.8, 42.8)
- moved C27 0.13 mm to (138.3, 45.6)
- moved C28 0.13 mm to (142.2, 45.6)
- moved Y2 0.13 mm to (140.2, 42.7)
- renumbered SW2 to SW1
Connections:
- U3 pad 13: unconnected-(U3-VBAT_OK-Pad13) -> Batt_ok
Routing:
- net Batt_ok: track 71.0 -> 94.6 mm, vias 4 -> 5
- net VCC: track 354.3 -> 347.1 mm
- net Net-(U3-VBAT_OV): track 20.8 -> 24.9 mm
- net Net-(U3-VREF_SAMP): track 8.33 -> 4.58 mm
- net Net-(U3-OK_HYST): track 37.3 -> 33.9 mm
- net Harvester_In: track 21.9 -> 24.7 mm
- net GND: track 162.8 -> 160.2 mm
- net Net-(J7-Pin_4): track 46.7 -> 45.5 mm
- net Net-(U3-VOC_SAMP): track 19.5 -> 20.6 mm
- net Net-(J7-Pin_3): track 43.8 -> 42.6 mm
Other:
- board text added: "m2"
