File: PassiveLiFiTag/LiFi_Receiver/LiFi_Receiver.kicad_sch (KiCad schematic)
At the start: 0 parts

Commit message: added updates
Changed lines of the file:
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@@
     (fill (type color) (color 235 234 255 1))
   )
-  (text "RH/T Sensors" (at 38.1 102.87 0)
+  (text "RH/T Sensors" (at 41.91 101.6 0)
     (effects (font (face "Ubuntu") (size 3 3)) (justify left bottom))
   )
-  (text "/Peripherals\n" (at 120.65 177.8 0)
+  (text "/Peripherals\n" (at 129.54 180.34 0)
     (effects (font (face "Ubuntu") (size 3 3)) (justify left bottom))
   )
-  (text "LiFi Comm Rx\n" (at 204.47 88.9 0)
+  (text "LiFi Comm Rx\n" (at 208.28 87.63 0)
     (effects (font (face "Ubuntu") (size 3 3)) (justify left bottom))
   )
-  (text "MSPFR5994\n" (at 127 107.95 0)
+  (text "MSPFR5994\n" (at 121.92 105.41 0)
     (effects (font (face "Ubuntu") (size 5 5)) (justify left bottom))
   )
-  (text "RF Backscatter\n" (at 123.19 35.56 0)
+  (text "RF Backscatter\n" (at 127 34.29 0)
     (effects (font (face "Ubuntu") (size 3 3)) (justify left bottom))
   )
-  (text "Buttons" (at 120.65 171.45 0)
+  (text "Buttons" (at 129.54 173.99 0)
     (effects (font (face "Ubuntu") (size 3 3)) (justify left bottom))
   )
-  (text "LiFi Power \n\n" (at 208.28 128.27 0)
+  (text "LiFi Power \n\n" (at 212.09 124.46 0)
     (effects (font (face "Ubuntu") (size 3 3)) (justify left bottom))
   )

Commit message: Added Updates
Other:
- sheet Peripherals renamed Battery Harvester_&_Peripherals
Changed lines of the file:
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@@
     (stroke (width 0.1524) (type solid))
     (fill (color 0 0 0 0.0000))
-    (property "Sheetname" "Peripherals" (at 12.7 230.4284 0)
+    (property "Sheetname" "Battery Harvester_&_Peripherals" (at 12.7 230.4284 0)
       (effects (font (size 1 1)) (justify left bottom))
     )
