File: PassiveLiFiTag/LiFi_Receiver/MSP430FR5994.kicad_sch (KiCad schematic)
At the start: 10 parts, among them U2 MSP430FR5994IPNR, Y1 Crystal_Small

Commit message: Continuing to update Hardware Design
Parts:
- renumbered C6 to C5, C5 to C6, U2 to U1
Connections:
- net UCB2SDA: now reaches U1.13 (P7.0_UCB2SIMO_UCB2SDA)
- net UCB2SCL: now reaches U1.14 (P7.1_UCB2SOMI_UCB2SCL)
Changed lines of the file:
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@@
+    (stroke (width 0) (type default))
+  )
+  (wire (pts (xy 39.37 116.84) (xy 59.69 116.84))
     (stroke (width 0) (type default))
   )
@@
   )
   (wire (pts (xy 50.8 25.4) (xy 50.8 27.94))
+    (stroke (width 0) (type default))
+  )
+  (wire (pts (xy 39.37 119.38) (xy 59.69 119.38))
     (stroke (width 0) (type default))
   )
@@
     )
   )
+  (global_label "UCB2SDA" (shape input) (at 39.37 116.84 180) (fields_autoplaced)
+    (effects (font (size 1.27 1.27)) (justify right))
+    (property "Intersheetrefs" "${INTERSHEET_REFS}" (at 27.7367 116.84 0)
+      (effects (font (size 1.27 1.27)) (justify right) hide)
+    )
+  )
   (global_label "AVCC_DVSS_" (shape input) (at 50.8 25.4 90) (fields_autoplaced)
     (effects (font (size 1 1)) (justify left))
@@
     )
   )
+  (global_label "UCB2SCL" (shape input) (at 39.37 119.38 180) (fields_autoplaced)
+    (effects (font (size 1.27 1.27)) (justify right))
+    (property "Intersheetrefs" "${INTERSHEET_REFS}" (at 27.7972 119.38 0)
+      (effects (font (size 1.27 1.27)) (justify right) hide)
+    )
+  )
   (global_label "P2.0_UART_TXD" (shape input) (at 187.96 27.94 0) (fields_autoplaced)
     (effects (font (size 1.27 1.27)) (justify left))
@@
   (symbol (lib_id "Device:C_Polarized_Small_US") (at 220.98 151.13 0) (unit 1)
     (in_bom yes) (on_board yes) (dnp no)
-    (property "Reference" "C6" (at 215.9 149.86 0)
+    (property "Reference" "C5" (at 215.9 149.86 0)
       (effects (font (size 1.27 1.27)) (justify left))
     )
@@
       (project "LiFi_Receiver"
         (path "/00b0bd1a-ca4b-4e13-a567-185f08cebf70/8a8bdf70-8118-4996-b9d8-1922bdfdf570"
-          (reference "C6") (unit 1)
+          (reference "C5") (unit 1)
         )
       )
@@
   (symbol (lib_id "Device:C_Small") (at 19.05 139.7 0) (unit 1)
     (in_bom yes) (on_board yes) (dnp no)
-    (property "Reference" "C5" (at 13.97 138.43 0)
+    (property "Reference" "C6" (at 13.97 138.43 0)
       (effects (font (size 1 1)) (justify left))
     )
@@
       (project "LiFi_Receiver"
         (path "/00b0bd1a-ca4b-4e13-a567-185f08cebf70/8a8bdf70-8118-4996-b9d8-1922bdfdf570"
-          (reference "C5") (unit 1)
+          (reference "C6") (unit 1)
         )
       )
@@
   (symbol (lib_id "LiFi_Receiver:MSP430FR5994IPNR") (at 146.05 91.44 0) (unit 1)
     (in_bom yes) (on_board yes) (dnp no) (fields_autoplaced)
-    (property "Reference" "U2" (at 146.05 17.78 0)
+    (property "Reference" "U1" (at 112.395 17.78 0)
       (effects (font (size 1 1)))
     )
-    (property "Value" "MSP430FR5994IPNR" (at 146.05 20.32 0)
+    (property "Value" "MSP430FR5994IPNR" (at 112.395 20.32 0)
       (effects (font (size 1 1)))
     )
@@
       (project "LiFi_Receiver"
         (path "/00b0bd1a-ca4b-4e13-a567-185f08cebf70/8a8bdf70-8118-4996-b9d8-1922bdfdf570"
-          (reference "U2") (unit 1)
-        )
-      )
+          (reference "U1") (unit 1)
+        )
+      )

Commit message: Added updates
Parts:
- C1, C2, C3, C4, C5, C6, C7: footprint (none) -> Capacitor_SMD:C_01005_0402Metric
- R1: footprint (none) -> Resistor_SMD:R_01005_0402Metric
- U1: footprint PN0080A_N -> Library:PN0080A_L
- Y1: footprint (none) -> Library:xtal-2
Changed lines of the file:
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@@
       (effects (font (size 1 1)) (justify left))
     )
-    (property "Footprint" "" (at 198.12 151.13 0)
+    (property "Footprint" "Capacitor_SMD:C_01005_0402Metric" (at 198.12 151.13 0)
       (effects (font (size 1 1)) hide)
     )
@@
       (effects (font (size 1 1)))
     )
-    (property "Footprint" "" (at 38.1 27.94 0)
+    (property "Footprint" "Resistor_SMD:R_01005_0402Metric" (at 38.1 27.94 0)
       (effects (font (size 1 1)) hide)
     )
@@
       (effects (font (size 1 1)) (justify left))
     )
-    (property "Footprint" "" (at 213.36 151.13 0)
+    (property "Footprint" "Capacitor_SMD:C_01005_0402Metric" (at 213.36 151.13 0)
       (effects (font (size 1 1)) hide)
     )
@@
       (effects (font (size 1 1)) (justify left))
     )
-    (property "Footprint" "" (at 205.74 151.13 0)
+    (property "Footprint" "Capacitor_SMD:C_01005_0402Metric" (at 205.74 151.13 0)
       (effects (font (size 1 1)) hide)
     )
@@
       (effects (font (size 1.27 1.27)) (justify left))
     )
-    (property "Footprint" "" (at 220.98 151.13 0)
+    (property "Footprint" "Capacitor_SMD:C_01005_0402Metric" (at 220.98 151.13 0)
       (effects (font (size 1.27 1.27)) hide)
     )
@@
       (effects (font (size 1.27 1.27)) hide)
     )
-    (property "Footprint" "" (at 24.13 148.59 0)
+    (property "Footprint" "Library:xtal-2" (at 24.13 148.59 0)
       (effects (font (size 1.27 1.27)) hide)
     )
@@
       (effects (font (size 1 1)) (justify left))
     )
-    (property "Footprint" "" (at 181.61 151.13 0)
+    (property "Footprint" "Capacitor_SMD:C_01005_0402Metric" (at 181.61 151.13 0)
       (effects (font (size 1 1)) hide)
     )
@@
       (effects (font (size 1 1)) (justify left))
     )
-    (property "Footprint" "" (at 29.21 139.7 0)
+    (property "Footprint" "Capacitor_SMD:C_01005_0402Metric" (at 29.21 139.7 0)
       (effects (font (size 1 1)) hide)
     )
@@
       (effects (font (size 1 1)) (justify left))
     )
-    (property "Footprint" "" (at 19.05 139.7 0)
+    (property "Footprint" "Capacitor_SMD:C_01005_0402Metric" (at 19.05 139.7 0)
       (effects (font (size 1 1)) hide)
     )
@@
       (effects (font (size 1 1)))
     )
-    (property "Footprint" "PN0080A_N" (at 146.05 91.44 0)
+    (property "Footprint" "Library:PN0080A_L" (at 146.05 91.44 0)
       (effects (font (size 1 1) italic) hide)
     )

Commit message: Added Updates
Parts:
- C5: footprint Capacitor_SMD:C_01005_0402Metric -> LIFI-FOOTPRINTS:TAJA_AVX-M
Changed lines of the file:
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@@
       (effects (font (size 1.27 1.27)) (justify left))
     )
-    (property "Footprint" "Capacitor_SMD:C_01005_0402Metric" (at 220.98 151.13 0)
+    (property "Footprint" "LIFI-FOOTPRINTS:TAJA_AVX-M" (at 220.98 151.13 0)
       (effects (font (size 1.27 1.27)) hide)
     )

Commit message: Added Updates
Changed lines of the file:
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@@
       (effects (font (size 1 1)) hide)
     )
-    (property "Value" "GND" (at 198.12 162.56 0)
-      (effects (font (size 1 1)))
+    (property "Value" "GND" (at 200.66 158.7499 0)
+      (effects (font (size 1 1)) (justify left))
     )
     (property "Footprint" "" (at 198.12 157.48 0)

Commit message: Design almost completed
Parts:
- added C27, C28: DNP, Capacitor_SMD:C_0603_1608Metric, symbol Device:C_Small
- added J6, J7: Conn_01x08, Connector_PinHeader_2.54mm:PinHeader_2x04_P2.54mm_Vertical, symbol Connector_Generic:Conn_01x08
- added TP3: SDA, TestPoint:TestPoint_Pad_D1.5mm, symbol Connector:TestPoint
- added TP4: SCL, TestPoint:TestPoint_Pad_D1.5mm, symbol Connector:TestPoint
- added Y2: Crystal_Small, Library:xtal-2, symbol Device:Crystal_Small
- C1, C2, C3, C4, C6, C7: footprint Capacitor_SMD:C_01005_0402Metric -> Capacitor_SMD:C_0603_1608Metric
- C5: footprint LIFI-FOOTPRINTS:TAJA_AVX-M -> Capacitor_SMD:C_0603_1608Metric
- R1: footprint Resistor_SMD:R_01005_0402Metric -> Resistor_SMD:R_0603_1608Metric
Connections:
- net GND: now also C27.1, C28.1
- net UCB2SCL: now also TP4.1
- net UCB2SDA: now also TP3.1
- net at U1.12 (P4.7): now also J7.1 (Pin_1)
- net at U1.31 (P4.0_A8): now also J7.8 (Pin_8)
- net at U1.32 (P4.1_A9): now also J7.7 (Pin_7)
- net at U1.33 (P4.2_A10): now also J7.6 (Pin_6)
- net at U1.34 (P4.3_A11): now also J7.5 (Pin_5)
- net at U1.53 (P5.0_UCB1SIMO_UCB1SDA): now also J6.1 (Pin_1)
- net at U1.54 (P5.1_UCB1SOMI_UCB1SCL): now also J6.2 (Pin_2)
- net at U1.55 (P5.2_UCB1CLK_TA4CLK): now also J6.3 (Pin_3)
- net at U1.56 (P5.3_UCB1STE): now also J6.4 (Pin_4)
- net at U1.57 (P4.4_TB0.5): now also J7.4 (Pin_4)
- net at U1.58 (P4.5): now also J7.3 (Pin_3)
- net at U1.59 (P4.6): now also J7.2 (Pin_2)
- net at U1.65 (P5.4_UCA2TXD_UCA2SIMO_TB0OUTH): now also J6.5 (Pin_5)
- net at U1.66 (P5.5_UCA2RXD_UCA2SOMI_ACLK): now also J6.6 (Pin_6)
- net at U1.67 (P5.6_UCA2CLK_TA4.0_SMCLK): now also J6.7 (Pin_7)
- net at U1.68 (P5.7_UCA2STE_TA4.1_MCLK): now also J6.8 (Pin_8)
- net at U1.74 (PJ.6_HFXIN): now also C28.2, Y2.2
- net at U1.75 (PJ.7_HFXOUT): now also C27.2, Y2.1
- no-connect marks 0 -> 44
Other:
- note added: "DNP"
