File: PassiveLiFiTag/LiFi_Receiver/RHT_Sensors.kicad_sch (KiCad schematic)
At the start: 0 parts

Commit message: Added some small peripherals and voltage supplies/decoupling caps
Parts:
- added J2: Conn_01x06, symbol Connector_Generic:Conn_01x06
- added R5: TC164-JR-072K2L, YAG_TC164_YAG, symbol LiFi_Receiver:TC164-JR-072K2L
- added U4, U5: HDC2080DMBR, DMB0006A, symbol LiFi_Receiver:HDC2080DMBR
Connections:
- new net GND: J2.6 (Pin_6), U4.2 (GND), U4.4 (DRDY_INT), U4.7 (PAD), U5.2 (GND), U5.3 (ADDR), U5.4 (DRDY_INT), U5.7 (PAD)
- new net SCL1_out: J2.2 (Pin_2), R5.2, U4.6 (SCL)
- new net SCL2_out: J2.4 (Pin_4), R5.4, U5.6 (SCL)
- new net SDA1_out: J2.3 (Pin_3), R5.1, U4.1 (SDA)
- new net SDA2_out: J2.5 (Pin_5), R5.3, U5.1 (SDA)
- new net VCC: J2.1 (Pin_1), R5.5, R5.6, R5.7, R5.8, U4.3 (ADDR), U4.5 (VDD), U5.5 (VDD)

Commit message: Continuing to update Hardware Design
Parts:
- removed J2: Conn_01x06, symbol Connector_Generic:Conn_01x06
- removed R5: TC164-JR-072K2L, YAG_TC164_YAG, symbol LiFi_Receiver:TC164-JR-072K2L
- added C11, C12: .1uF, symbol Device:C_Small
- added RN1: 742C083472JP, , symbol LifiLib:742C083472JP
Connections:
- net SCL2_out is gone; now on net UCB2SCL: U5.6 (SCL)
- net SDA2_out is gone; now on net UCB2SDA: U5.1 (SDA)
- net GND: now also C11.2, C12.2
- net VCC: now also C11.1, C12.1, RN1.4
- net SCL1_out renamed UCB2SCL
- net UCB2SCL: now also RN1.5
- net SDA1_out renamed UCB2SDA
- net UCB2SDA: now also RN1.5

Commit message: added updates
Parts:
- added NT1, NT2, NT3, NT4: NetTie_3, symbol Device:NetTie_3
- C11, C12: footprint (none) -> Capacitor_SMD:C_01005_0402Metric
- RN1: footprint (none) -> LIFI-FOOTPRINTS:Res_network
- U4, U5: footprint DMB0006A -> LIFI-FOOTPRINTS:HDC2080_1
Connections:
- net GND: no longer U4.7 (PAD), U5.7 (PAD)
- net UCB2SCL: now also NT1.2, NT4.2; no longer RN1.5, U4.6 (SCL), U5.6 (SCL)
- net UCB2SDA: now also NT2.2, NT3.2; no longer RN1.5, U4.1 (SDA), U5.1 (SDA)
- new net: NT4.3, U4.6 (SCL)
- new net: NT1.3, U5.6 (SCL)
- new net: NT3.3, U4.1 (SDA)
- new net: NT2.3, U5.1 (SDA)
- new net scl1: NT4.1, RN1.5
- new net scl2: NT1.1, RN1.5
- new net sda1: NT3.1, RN1.5
- new net sda2: NT2.1, RN1.5
- no-connect marks 0 -> 2

Commit message: Added Updates
Parts:
- added JP1, JP2, JP3: SolderJumper_2_Open, Jumper:SolderJumper-2_P1.3mm_Open_TrianglePad1.0x1.5mm, symbol Jumper:SolderJumper_2_Open
Connections:
- net VCC: now also JP3.1 (A); no longer C12.1, U5.5 (VDD)
- net scl2: now also JP2.2 (B); no longer RN1.5
- net sda2: now also JP1.1 (A); no longer RN1.5
- new net: JP2.1 (A), RN1.5
- new net: JP1.2 (B), RN1.5
- new net: C12.1, JP3.2 (B), U5.5 (VDD)
Changed lines of the file:
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@@
+    (stroke (width 0) (type default))
+  )
+  (wire (pts (xy 142.24 120.65) (xy 142.24 124.46))
     (stroke (width 0) (type default))
   )
@@
     (stroke (width 0) (type default))
   )
-  (wire (pts (xy 146.05 120.65) (xy 154.94 120.65))
+  (wire (pts (xy 142.24 120.65) (xy 154.94 120.65))
     (stroke (width 0) (type default))
   )
@@
     (stroke (width 0) (type default))
   )
-  (wire (pts (xy 147.32 49.53) (xy 152.4 49.53))
+  (wire (pts (xy 132.08 49.53) (xy 152.4 49.53))
+    (stroke (width 0) (type default))
+  )
+  (wire (pts (xy 132.08 46.99) (xy 152.4 46.99))
     (stroke (width 0) (type default))
   )
@@
     (stroke (width 0) (type default))
   )
+  (wire (pts (xy 146.05 97.79) (xy 146.05 102.87))
+    (stroke (width 0) (type default))
+  )
   (wire (pts (xy 190.5 113.03) (xy 200.66 113.03))
     (stroke (width 0) (type default))
@@
     (stroke (width 0) (type default))
   )
-  (wire (pts (xy 147.32 46.99) (xy 152.4 46.99))
-    (stroke (width 0) (type default))
-  )
   (wire (pts (xy 60.96 120.65) (xy 60.96 110.49))
     (stroke (width 0) (type default))
@@
     (stroke (width 0) (type default))
   )
-  (wire (pts (xy 146.05 120.65) (xy 146.05 132.08))
-    (stroke (width 0) (type default))
-  )
-  (wire (pts (xy 146.05 106.68) (xy 146.05 110.49))
+  (wire (pts (xy 121.92 49.53) (xy 124.46 49.53))
+    (stroke (width 0) (type default))
+  )
+  (wire (pts (xy 121.92 46.99) (xy 124.46 46.99))
     (stroke (width 0) (type default))
   )
@@
     (effects (font (size 1.27 1.27)) (justify left top))
   )
-  (text_box "I2C pullups\n"
-    (at 88.9 16.51 0) (size 133.35 55.88)
-    (stroke (width 0) (type default))
-    (fill (type none))
-    (effects (font (size 1.27 1.27)) (justify left top))
-  )
-  (global_label "sda2" (shape input) (at 147.32 46.99 180) (fields_autoplaced)
-    (effects (font (size 1.27 1.27)) (justify right))
-    (property "Intersheetrefs" "${INTERSHEET_REFS}" (at 139.7992 46.99 0)
+  (global_label "sda2" (shape input) (at 121.92 46.99 180) (fields_autoplaced)
+    (effects (font (size 1.27 1.27)) (justify right))
+    (property "Intersheetrefs" "${INTERSHEET_REFS}" (at 114.3992 46.99 0)
       (effects (font (size 1.27 1.27)) (justify right) hide)
     )
@@
     )
   )
-  (global_label "scl2" (shape input) (at 147.32 49.53 180) (fields_autoplaced)
-    (effects (font (size 1.27 1.27)) (justify right))
-    (property "Intersheetrefs" "${INTERSHEET_REFS}" (at 140.3434 49.53 0)
+  (global_label "scl2" (shape input) (at 121.92 49.53 180) (fields_autoplaced)
+    (effects (font (size 1.27 1.27)) (justify right))
+    (property "Intersheetrefs" "${INTERSHEET_REFS}" (at 114.9434 49.53 0)
       (effects (font (size 1.27 1.27)) (justify right) hide)
     )
@@
     )
   )
-  (symbol (lib_id "power:VCC") (at 146.05 106.68 0) (unit 1)
-    (in_bom yes) (on_board yes) (dnp no) (fields_autoplaced)
-    (property "Reference" "#2.4FromReg0102" (at 146.05 110.49 0)
-      (effects (font (size 1.27 1.27)) hide)
-    )
-    (property "Value" "VCC" (at 146.05 101.6 0)
-      (effects (font (size 1.27 1.27)))
-    )
-    (property "Footprint" "" (at 146.05 106.68 0)
-      (effects (font (size 1.27 1.27)) hide)
-    )
-    (property "Datasheet" "" (at 146.05 106.68 0)
+  (symbol (lib_id "Jumper:SolderJumper_2_Open") (at 128.27 49.53 180) (unit 1)
+    (in_bom yes) (on_board yes) (dnp no)
+    (property "Reference" "JP2" (at 128.27 53.34 0)
+      (effects (font (size 1.27 1.27)))
+    )
+    (property "Value" "SolderJumper_2_Open" (at 128.27 55.88 0)
+      (effects (font (size 1.27 1.27)))
+    )
+    (property "Footprint" "Jumper:SolderJumper-2_P1.3mm_Open_TrianglePad1.0x1.5mm" (at 128.27 49.53 0)
+      (effects (font (size 1.27 1.27)) hide)
+    )
+    (property "Datasheet" "~" (at 128.27 49.53 0)
+      (effects (font (size 1.27 1.27)) hide)
+    )
+    (pin "2")
+    (pin "1")
+    (instances
+      (project "LiFi_Receiver"
+        (path "/00b0bd1a-ca4b-4e13-a567-185f08cebf70/b5c5dd7e-aaeb-4581-8f1f-2825f847a429"
+          (reference "JP2") (unit 1)
+        )
+      )
+    )
+  )
+  (symbol (lib_id "power:VCC") (at 146.05 97.79 0) (unit 1)
+    (in_bom yes) (on_board yes) (dnp no) (fields_autoplaced)
+    (property "Reference" "#2.4FromReg0102" (at 146.05 101.6 0)
+      (effects (font (size 1.27 1.27)) hide)
+    )
+    (property "Value" "VCC" (at 146.05 92.71 0)
+      (effects (font (size 1.27 1.27)))
+    )
+    (property "Footprint" "" (at 146.05 97.79 0)
+      (effects (font (size 1.27 1.27)) hide)
+    )
+    (property "Datasheet" "" (at 146.05 97.79 0)
       (effects (font (size 1.27 1.27)) hide)
     )
@@
     )
   )
-  (symbol (lib_id "power:GND") (at 146.05 132.08 0) (unit 1)
-    (in_bom yes) (on_board yes) (dnp no) (fields_autoplaced)
-    (property "Reference" "#PWR011" (at 146.05 138.43 0)
-      (effects (font (size 1.27 1.27)) hide)
-    )
-    (property "Value" "GND" (at 146.05 137.16 0)
-      (effects (font (size 1.27 1.27)))
-    )
-    (property "Footprint" "" (at 146.05 132.08 0)
-      (effects (font (size 1.27 1.27)) hide)
-    )
-    (property "Datasheet" "" (at 146.05 132.08 0)
+  (symbol (lib_id "Jumper:SolderJumper_2_Open") (at 146.05 106.68 270) (unit 1)
+    (in_bom yes) (on_board yes) (dnp no)
+    (property "Reference" "JP3" (at 142.24 104.14 90)
+      (effects (font (size 1.27 1.27)))
+    )
+    (property "Value" "SolderJumper_2_Open" (at 161.29 153.67 90)
+      (effects (font (size 1.27 1.27)) hide)
+    )
+    (property "Footprint" "Jumper:SolderJumper-2_P1.3mm_Open_TrianglePad1.0x1.5mm" (at 146.05 106.68 0)
+      (effects (font (size 1.27 1.27)) hide)
+    )
+    (property "Datasheet" "~" (at 146.05 106.68 0)
+      (effects (font (size 1.27 1.27)) hide)
+    )
+    (pin "2")
+    (pin "1")
+    (instances
+      (project "LiFi_Receiver"
+        (path "/00b0bd1a-ca4b-4e13-a567-185f08cebf70/b5c5dd7e-aaeb-4581-8f1f-2825f847a429"
+          (reference "JP3") (unit 1)
+        )
+      )
+    )
+  )
+  (symbol (lib_id "power:GND") (at 142.24 124.46 0) (unit 1)
+    (in_bom yes) (on_board yes) (dnp no) (fields_autoplaced)
+    (property "Reference" "#PWR011" (at 142.24 130.81 0)
+      (effects (font (size 1.27 1.27)) hide)
+    )
+    (property "Value" "GND" (at 142.24 129.54 0)
+      (effects (font (size 1.27 1.27)))
+    )
+    (property "Footprint" "" (at 142.24 124.46 0)
+      (effects (font (size 1.27 1.27)) hide)
+    )
+    (property "Datasheet" "" (at 142.24 124.46 0)
       (effects (font (size 1.27 1.27)) hide)
     )
@@
         )
       )
+    )
+  )
+  (symbol (lib_id "Jumper:SolderJumper_2_Open") (at 128.27 46.99 0) (unit 1)
+    (in_bom yes) (on_board yes) (dnp no) (fields_autoplaced)
+    (property "Reference" "JP1" (at 128.27 40.64 0)
+      (effects (font (size 1.27 1.27)))
+    )
+    (property "Value" "SolderJumper_2_Open" (at 128.27 43.18 0)
+      (effects (font (size 1.27 1.27)))
+    )
+    (property "Footprint" "Jumper:SolderJumper-2_P1.3mm_Open_TrianglePad1.0x1.5mm" (at 128.27 46.99 0)
+      (effects (font (size 1.27 1.27)) hide)
+    )
+    (property "Datasheet" "~" (at 128.27 46.99 0)
+      (effects (font (size 1.27 1.27)) hide)
+    )
+    (pin "2")
+    (pin "1")
+    (instances
+      (project "LiFi_Receiver"
+        (path "/00b0bd1a-ca4b-4e13-a567-185f08cebf70/b5c5dd7e-aaeb-4581-8f1f-2825f847a429"
+          (reference "JP1") (unit 1)
+        )
+      )

Commit message: Added Updates
Changed lines of the file:
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@@
+    (effects (font (size 1.27 1.27)) (justify left top))
+  )
+  (text_box "Pull-Up Array\n\n"
+    (at 19.05 15.24 0) (size 259.08 55.88)
+    (stroke (width 0) (type default))
+    (fill (type none))
     (effects (font (size 1.27 1.27)) (justify left top))
   )

Commit message: Design almost completed
Parts:
- removed NT1, NT2, NT3, NT4: NetTie_3, symbol Device:NetTie_3
- C11, C12: footprint Capacitor_SMD:C_01005_0402Metric -> Capacitor_SMD:C_0603_1608Metric
- RN1: footprint LIFI-FOOTPRINTS:Res_network -> Library:RESCAV80P320X160X70-8N
- U4, U5: footprint LIFI-FOOTPRINTS:HDC2080_1 -> Library:DMB0006A_NV
Connections:
- net scl1 is gone; now on net VCC: RN1.5 (4)
- net scl2 is gone; now on net UCB2SCL: JP2.2 (B)
- net sda1 is gone; now on net VCC: RN1.5 (4)
- net sda2 is gone; now on net UCB2SDA_BYP: JP1.1 (A)
- net UCB2SCL: now also RN1.2 (5), U4.6 (SCL)
- net UCB2SDA: now also JP1.2 (B), RN1.1 (5), U4.1 (SDA)
- net VCC: now also RN1.6 (4), RN1.7 (4), RN1.8 (4); no longer RN1.4
- net UCB2SCL_BYP: now reaches U5.6 (SCL)
- net UCB2SCL_BYP: now also JP2.1 (A), RN1.4 (5)
- net UCB2SDA_BYP: now reaches U5.1 (SDA)
- net UCB2SDA_BYP: now also RN1.3 (5)
Other:
- moved on the sheet: RN1
