File: PassiveLiFiTag/LiFi_Receiver/ReceiverAndPower.kicad_sch (KiCad schematic)
At the start: 0 parts

Commit message: Added some small peripherals and voltage supplies/decoupling caps
Parts:
- added B1, B2, B3, B4: SM141K08TFV, SM141K08TFV_AAR, symbol LiFi_Receiver:SM141K08TFV
- added C8, C9: C_Small, symbol Device:C_Small
- added R2, R3: R_Small_US, symbol Device:R_Small_US
- added U1: TS881ILT, SOT23-5_TS881_TEX, symbol LiFi_Receiver:TS881ILT
- added U3: BQ25570RGRR, RGR0020A, symbol LiFi_Receiver:BQ25570RGRR
Connections:
- new net: C8.2, R2.1, U1.3 (IN+)
- new net Comparator Out: U1.1 (OUT)
- new net GND: C9.2, R2.2, U1.2 (VCC-), U1.4 (IN-)
- new net Harvester_In: C9.1, R3.2
- new net PV Out: C8.1, R3.1
- new net VCC: U1.5 (VCC+)
Other:
- note added: "* Need to Decide on Filter Values"

Commit message: Continuing to update Hardware Design
Parts:
- renumbered U1 to U2
Other:
- moved on the sheet: B1, B2, B3, B4, C8, C9, R2, R3, U2, U3

Commit message: updating changes
Parts:
- added C13, C14, C15, C16, C17: .1uF, symbol Device:C_Small
- added U10, U8, U9: ADG721BRMZ-REEL, RM_8_ADI, symbol LiFi_Receiver:ADG721BRMZ-REEL
- added U6, U7: ADG722BRMZ-REEL7, RM_8_ADI, symbol LiFi_Receiver:ADG722BRMZ-REEL7
Connections:
- net GND: now also C13.2, C14.2, C15.2, C16.2, C17.2, U10.4 (GND), U6.4 (GND), U7.4 (GND), U8.4 (GND), U9.4 (GND)
- net VCC: now also C13.1, C14.1, C15.1, C16.1, C17.1, U10.8 (VDD), U6.8 (VDD), U7.8 (VDD), U8.8 (VDD), U9.8 (VDD)
- net P2+: now reaches B2.1
- net P2+: now also U6.2 (D1), U8.2 (D1), U8.5 (S2)
- net P2-: now reaches B2.2
- net P2-: now also U10.1 (S1), U6.5 (S2), U9.6 (D2)
- net P3+: now reaches B3.1
- net P3+: now also U6.6 (D2), U8.6 (D2), U9.1 (S1)
- net P3-: now reaches B3.2
- net P3-: now also U10.2 (D1), U10.5 (S2), U7.1 (S1)
- net P1+: now reaches B1.1
- net P1+: now also U8.1 (S1)
- net P1-: now reaches B1.2
- net P1-: now also U6.1 (S1), U9.5 (S2)
- net P4+: now reaches B4.1
- net P4+: now also U7.2 (D1), U9.2 (D1)
- net P4-: now reaches B4.2
- net P4-: now also U10.6 (D2)
- new net Batt_ok: U10.3 (IN2), U10.7 (IN1), U6.3 (IN2), U6.7 (IN1), U7.3 (IN2), U7.7 (IN1), U8.3 (IN2), U8.7 (IN1), U9.3 (IN2), U9.7 (IN1)
- no-connect marks 0 -> 2
Other:
- moved on the sheet: B1, B2, B3, B4, U3

Commit message: added Updates
Parts:
- C13, C14, C15, C16, C17: footprint (none) -> Capacitor_SMD:C_01005_0402Metric
Changed lines of the file:
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@@
       (effects (font (size 1.27 1.27)) (justify right))
     )
-    (property "Footprint" "" (at 149.86 34.29 0)
+    (property "Footprint" "Capacitor_SMD:C_01005_0402Metric" (at 149.86 34.29 0)
       (effects (font (size 1.27 1.27)) hide)
     )
@@
       (effects (font (size 1.27 1.27)) (justify right))
     )
-    (property "Footprint" "" (at 109.22 109.22 0)
+    (property "Footprint" "Capacitor_SMD:C_01005_0402Metric" (at 109.22 109.22 0)
       (effects (font (size 1.27 1.27)) hide)
     )
@@
       (effects (font (size 1.27 1.27)) (justify right))
     )
-    (property "Footprint" "" (at 149.86 63.5 0)
+    (property "Footprint" "Capacitor_SMD:C_01005_0402Metric" (at 149.86 63.5 0)
       (effects (font (size 1.27 1.27)) hide)
     )
@@
       (effects (font (size 1.27 1.27)) (justify right))
     )
-    (property "Footprint" "" (at 109.22 171.45 0)
+    (property "Footprint" "Capacitor_SMD:C_01005_0402Metric" (at 109.22 171.45 0)
       (effects (font (size 1.27 1.27)) hide)
     )
@@
       (effects (font (size 1.27 1.27)) (justify right))
     )
-    (property "Footprint" "" (at 109.22 140.97 0)
-      (effects (font (size 1.27 1.27)) hide)
-    )
+    (property "Footprint" "Capacitor_SMD:C_01005_0402Metric" (at 109.22 140.97 0)
+      (effects (font (size 1.27 1.27)) hide)
+    )

Commit message: added updates
Parts:
- removed B1, B2, B3, B4: SM141K08TFV, SM141K08TFV_AAR, symbol LiFi_Receiver:SM141K08TFV
- added J2, J3, J4, J5: Conn_01x02, Connector_PinSocket_2.54mm:PinSocket_1x02_P2.54mm_Vertical, symbol Connector_Generic:Conn_01x02
- U10, U6, U7, U8, U9: footprint RM_8_ADI -> LIFI-FOOTPRINTS:RM_8_ADI-M
Connections:
- net P1+: now also J2.1 (Pin_1)
- net P1-: now also J2.2 (Pin_2)
- net P2+: now also J3.1 (Pin_1)
- net P2-: now also J3.2 (Pin_2)
- net P3+: now also J4.1 (Pin_1)
- net P3-: now also J4.2 (Pin_2)
- net P4+: now also J5.1 (Pin_1)
- net P4-: now also J5.2 (Pin_2)

Commit message: Added updates
Parts:
- C8, C9: footprint (none) -> Capacitor_SMD:C_0402_1005Metric
- R2, R3: footprint (none) -> Resistor_SMD:R_0402_1005Metric
- U2: footprint SOT23-5_TS881_TEX -> LIFI-FOOTPRINTS:TS88_3
Connections:
- net P4- is gone; now on net GND: J5.2 (Pin_2), U10.6 (D2)
- net PV Out is gone; now on net P1+: C8.1, R3.1
Changed lines of the file:
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@@
     (effects (font (size 2 2)) (justify left bottom))
   )
-  (global_label "PV Out" (shape input) (at 271.78 39.37 0) (fields_autoplaced)
-    (effects (font (size 1.27 1.27)) (justify left))
-    (property "Intersheetrefs" "${INTERSHEET_REFS}" (at 281.2966 39.37 0)
+  (global_label "V_Plus" (shape input) (at 271.78 39.37 0) (fields_autoplaced)
+    (effects (font (size 1.27 1.27)) (justify left))
+    (property "Intersheetrefs" "${INTERSHEET_REFS}" (at 280.9337 39.37 0)
       (effects (font (size 1.27 1.27)) (justify left) hide)
     )
@@
     (effects (font (size 1.27 1.27)) (justify left))
     (property "Intersheetrefs" "${INTERSHEET_REFS}" (at 101.0171 175.26 0)
-      (effects (font (size 1.27 1.27)) (justify left) hide)
-    )
-  )
-  (global_label "V_Minus" (shape input) (at 71.12 77.47 0) (fields_autoplaced)
-    (effects (font (size 1.27 1.27)) (justify left))
-    (property "Intersheetrefs" "${INTERSHEET_REFS}" (at 81.5437 77.47 0)
       (effects (font (size 1.27 1.27)) (justify left) hide)
     )
@@
       (effects (font (size 1.27 1.27)))
     )
-    (property "Footprint" "" (at 264.16 26.67 0)
+    (property "Footprint" "Resistor_SMD:R_0402_1005Metric" (at 264.16 26.67 0)
       (effects (font (size 1.27 1.27)) hide)
     )
@@
       (effects (font (size 1.27 1.27)) (justify left))
     )
-    (property "Footprint" "" (at 256.54 55.88 0)
+    (property "Footprint" "Resistor_SMD:R_0402_1005Metric" (at 256.54 55.88 0)
       (effects (font (size 1.27 1.27)) hide)
     )
@@
         (path "/00b0bd1a-ca4b-4e13-a567-185f08cebf70/c6993dd6-5c17-4cc4-9f69-1140d0f1d252"
           (reference "C13") (unit 1)
+        )
+      )
+    )
+  )
+  (symbol (lib_id "power:GND") (at 71.12 77.47 0) (unit 1)
+    (in_bom yes) (on_board yes) (dnp no) (fields_autoplaced)
+    (property "Reference" "#PWR026" (at 71.12 83.82 0)
+      (effects (font (size 1.27 1.27)) hide)
+    )
+    (property "Value" "GND" (at 71.12 82.55 0)
+      (effects (font (size 1.27 1.27)))
+    )
+    (property "Footprint" "" (at 71.12 77.47 0)
+      (effects (font (size 1.27 1.27)) hide)
+    )
+    (property "Datasheet" "" (at 71.12 77.47 0)
+      (effects (font (size 1.27 1.27)) hide)
+    )
+    (pin "1")
+    (instances
+      (project "LiFi_Receiver"
+        (path "/00b0bd1a-ca4b-4e13-a567-185f08cebf70/c6993dd6-5c17-4cc4-9f69-1140d0f1d252"
+          (reference "#PWR026") (unit 1)
         )
       )
@@
       (effects (font (size 1.27 1.27)))
     )
-    (property "Footprint" "" (at 264.16 52.07 0)
+    (property "Footprint" "Capacitor_SMD:C_0402_1005Metric" (at 264.16 52.07 0)
       (effects (font (size 1.27 1.27)) hide)
     )
@@
       (effects (font (size 1.27 1.27)) (justify left))
     )
-    (property "Footprint" "" (at 259.08 31.75 0)
+    (property "Footprint" "Capacitor_SMD:C_0402_1005Metric" (at 259.08 31.75 0)
       (effects (font (size 1.27 1.27)) hide)
     )
@@
       (effects (font (size 1.524 1.524)))
     )
-    (property "Footprint" "SOT23-5_TS881_TEX" (at 207.01 38.1 0)
+    (property "Footprint" "LIFI-FOOTPRINTS:TS88_3" (at 207.01 38.1 0)
       (effects (font (size 1.27 1.27) italic) hide)
     )

Commit message: Added Updates
Parts:
- removed U3: BQ25570RGRR, RGR0020A, symbol LiFi_Receiver:BQ25570RGRR
- added C18, C19: C_Small, Connector_PinSocket_2.54mm:PinSocket_1x02_P2.54mm_Vertical, symbol Device:C_Small
- added JP5, JP6: Jumper_3_Open, Connector_PinHeader_2.54mm:PinHeader_1x03_P2.54mm_Vertical, symbol Jumper:Jumper_3_Open
- added R5, R6: R_Small_US, Connector_PinSocket_2.54mm:PinSocket_1x02_P2.54mm_Vertical, symbol Device:R_Small_US
Connections:
- net GND: now also C18.2, R6.2
- net Harvester_In: now also JP5.2 (C); no longer C9.1, R3.2
- net P1+: now also C19.1, R5.1
- net at C8.2, R2.1: now also JP6.3 (B); no longer U2.3 (IN+)
- new net: C9.1, JP5.1 (A), R3.2
- new net: C18.1, JP5.3 (B), R5.2
- new net: C19.2, JP6.1 (A), R6.1
- new net Comparator_In: JP6.2 (C), U2.3 (IN+)
Other:
- note removed: "* Need to Decide on Filter Values"
- moved on the sheet: C8, C9, R2, R3, U2

Commit message: Design almost completed
Parts:
- C13, C14, C15, C16, C17: footprint Capacitor_SMD:C_01005_0402Metric -> Capacitor_SMD:C_0603_1608Metric
- C8, C9: footprint Capacitor_SMD:C_0402_1005Metric -> Capacitor_SMD:C_0603_1608Metric
- R2, R3: footprint Resistor_SMD:R_0402_1005Metric -> Resistor_SMD:R_0603_1608Metric
- U10, U8, U9: footprint LIFI-FOOTPRINTS:RM_8_ADI-M -> Library:RM_8_ADI
- U2: footprint LIFI-FOOTPRINTS:TS88_3 -> Library:SOT23-5_TS881_TEX
- U6, U7: footprint LIFI-FOOTPRINTS:RM_8_ADI-M -> Library:RM_8_ADI-M
Other:
- moved on the sheet: C18, C19, C8, C9, JP5, JP6, R2, R3, R5, R6, U2
