File: PassiveLiFiTag/LiFi_Receiver/Peripherals.kicad_sch (KiCad schematic)
At the start: 0 parts

Commit message: Added some small peripherals and voltage supplies/decoupling caps
Parts:
- added C10: 1n, symbol Device:C_Small
- added J1: Conn_01x07, symbol Connector_Generic:Conn_01x07
- added R4: 27K, symbol Device:R_Small_US
- added SW1: SW_Push, symbol Switch:SW_Push
Connections:
- new net +3.3V: J1.3 (Pin_3)
- new net GND: C10.2, J1.1 (Pin_1), SW1.1
- new net P2.0_UART_TXD: J1.5 (Pin_5)
- new net P2.1_UART_RXD: J1.4 (Pin_4)
- new net TEST_SBWTCK: J1.7 (Pin_7)
- new net VCC: R4.1
- new net ~{RST}/SBWTDIO_N: C10.1, J1.6 (Pin_6), R4.2, SW1.2

Commit message: Added updates
Parts:
- SW1: footprint (none) -> Library:SW_TL59NF160Q
Changed lines of the file:
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@@
       (effects (font (size 1.27 1.27)))
     )
-    (property "Footprint" "" (at 241.3 34.29 0)
+    (property "Footprint" "Library:SW_TL59NF160Q" (at 241.3 34.29 0)
       (effects (font (size 1.27 1.27)) hide)
     )

Commit message: added updates
Parts:
- C10: footprint (none) -> Capacitor_SMD:C_01005_0402Metric
- R4: footprint (none) -> Resistor_SMD:R_01005_0402Metric
- SW1: footprint Library:SW_TL59NF160Q -> LIFI-FOOTPRINTS:SW_TL59NF160Q
Changed lines of the file:
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@@
       (effects (font (size 1.27 1.27)) (justify left))
     )
-    (property "Footprint" "" (at 252.73 44.45 0)
+    (property "Footprint" "Capacitor_SMD:C_01005_0402Metric" (at 252.73 44.45 0)
       (effects (font (size 1.27 1.27)) hide)
     )
@@
       (effects (font (size 1.27 1.27)))
     )
-    (property "Footprint" "Library:SW_TL59NF160Q" (at 241.3 34.29 0)
+    (property "Footprint" "LIFI-FOOTPRINTS:SW_TL59NF160Q" (at 241.3 34.29 0)
       (effects (font (size 1.27 1.27)) hide)
     )
@@
       (effects (font (size 1.27 1.27)) (justify left))
     )
-    (property "Footprint" "" (at 252.73 31.75 0)
+    (property "Footprint" "Resistor_SMD:R_01005_0402Metric" (at 252.73 31.75 0)
       (effects (font (size 1.27 1.27)) hide)
     )

Commit message: Added updates
Parts:
- J1: footprint (none) -> Connector_PinSocket_2.54mm:PinSocket_1x07_P2.54mm_Vertical
Connections:
- no-connect marks 0 -> 1
Changed lines of the file:
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@@
   (junction (at 252.73 39.37) (diameter 0) (color 0 0 0 0)
   )
+  (no_connect (at 260.35 71.12))
   (wire (pts (xy 252.73 34.29) (xy 252.73 39.37))
     (stroke (width 0) (type default))
@@
       (effects (font (size 1.27 1.27)) (justify left))
     )
-    (property "Footprint" "" (at 265.43 76.2 0)
-      (effects (font (size 1.27 1.27)) hide)
-    )
+    (property "Footprint" "Connector_PinSocket_2.54mm:PinSocket_1x07_P2.54mm_Vertical" (at 265.43 76.2 0)
+      (effects (font (size 1.27 1.27)) hide)
+    )

Commit message: Added Updates
Parts:
- added C20, C24: 4.7uF, Capacitor_SMD:C_01005_0402Metric, symbol Device:C_Small
- added C21, C25, C26: 0.1uF, Capacitor_SMD:C_01005_0402Metric, symbol Device:C_Small
- added C22: 22uF, Capacitor_SMD:C_01005_0402Metric, symbol Device:C_Small
- added C23: 0.01uF, Capacitor_SMD:C_01005_0402Metric, symbol Device:C_Small
- added L1: 22uH, Inductor_SMD:L_01005_0402Metric, symbol Device:L_Small
- added L2: 4.7uH, Inductor_SMD:L_01005_0402Metric, symbol Device:L_Small
- added R10, R11, R12, R13, R7, R8, R9: R_Small_US, Resistor_SMD:R_01005_0402Metric, symbol Device:R_Small_US
- added U11: S-1313B24-M5T1U3, Package_TO_SOT_SMD:SOT-23-5, symbol LifiLib:S-1313B24-M5T1U3
- added U3: BQ25570RGRR, Library:Bat_Harv2, symbol LiFi_Receiver:BQ25570RGRR
Connections:
- net GND: now also C20.2, C21.2, C22.2, C23.2, C24.2, C25.2, C26.2, R11.2, R13.2, R8.2, U11.2 (Vss), U3.1 (VSS), U3.15 (VSS), U3.17 (NC), U3.21 (PAD), U3.9 (NC)
- net VCC: now also C26.1, U11.5 (Vout)
- new net: R7.2, R8.1, U3.7 (VBAT_OV)
- new net: L2.2, U3.16 (LBUCK)
- new net: R10.2, R11.1, U3.11 (OK_PROG)
- new net: R12.1, R7.1, R9.1, U3.8 (VRDIV)
- new net: R12.2, R13.1, U3.12 (VOUT_SET)
- new net: C20.1, C21.1, U3.19 (VSTOR), U3.3 (VOC_SAMP)
- new net: L1.1, U3.20 (LBOOST)
- new net: C23.1, U3.4 (VREF_SAMP)
- new net: R10.1, R9.2, U3.10 (OK_HYST)
- new net Bat: U3.18 (VBAT)
- new net Harvester_In: C24.1, L1.2, U3.2 (VIN_DC)
- new net Harvester_out: C22.1, C25.1, L2.1, U11.1 (Vin), U11.3 (On/Off), U3.14 (VOUT)

Commit message: Design almost completed
Parts:
- removed SW1: SW_Push, LIFI-FOOTPRINTS:SW_TL59NF160Q, symbol Switch:SW_Push
- added H1, H2: MountingHole, MountingHole:MountingHole_2.2mm_M2, symbol Mechanical:MountingHole
- added J9: Conn_01x02, Connector_PinSocket_2.54mm:PinSocket_1x02_P2.54mm_Vertical, symbol Connector_Generic:Conn_01x02
- added SW2: PTS645SL43SMTR92LFS, Library:PTS645SL43SMTR92LFS_CNK-M, symbol LifiLib:PTS645SL43SMTR92LFS
- added TP1, TP2: TestPoint, TestPoint:TestPoint_Pad_D1.5mm, symbol Connector:TestPoint
- added TP5: 2.4v, TestPoint:TestPoint_Pad_D1.5mm, symbol Connector:TestPoint
- C10, C20, C21, C22, C23, C24, C25, C26: footprint Capacitor_SMD:C_01005_0402Metric -> Capacitor_SMD:C_0603_1608Metric
- L1, L2: footprint Inductor_SMD:L_01005_0402Metric -> Inductor_SMD:L_0603_1608Metric
- R10, R11, R12, R13, R4, R7, R8, R9: footprint Resistor_SMD:R_01005_0402Metric -> Resistor_SMD:R_0603_1608Metric
- U3: footprint Library:Bat_Harv2 -> Library:Bat_Harv1
Connections:
- net +3.3V is gone; now on net VCC: J1.3 (Pin_3)
- net Bat: now also J9.1 (Pin_1), TP1.1
- net GND: now also U3.5 (EN_N), J9.2 (Pin_2), SW2.1, SW2.2, TP2.1
- net VCC: now also TP5.1
- net ~{RST}/SBWTDIO_N: now also SW2.3, SW2.4
- no-connect marks 1 -> 2
Other:
- moved on the sheet: C10, C20, C21, C22, C23, C24, C26, J1, L1, L2, R10, R11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

Commit message: ready for design review
Connections:
- net Batt_ok: now reaches U3.13 (VBAT_OK)
Changed lines of the file:
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@@
+    )
+  )
+  (global_label "Batt_ok" (shape input) (at 74.93 68.58 180) (fields_autoplaced)
+    (effects (font (size 1.27 1.27)) (justify right))
+    (property "Intersheetrefs" "${INTERSHEET_REFS}" (at 64.9297 68.58 0)
+      (effects (font (size 1.27 1.27)) (justify right) hide)
     )
   )
